File: Lagopus_Board/Lagopus_A.sch (EAGLE design)
At the start: 39 parts, among them J1 PTH, J2 PTH, U1 MLX90614_, U2 VL53L1X, U3 APDS-9301, U5 AS72652, U6 AS72651, U7 AS72653, U8 MX25L4006E

Commit message: Ordered Version 1.0 from Seeed
Lemming_SMD V1.0
Lagopus_A V1.0
Lagopus_B V1.0
Parts:
- removed C7: 1.0uF, SparkFun-Capacitors:1.0UF-0603-16V-10%
- removed C8, C9: 10uF, SparkFun-Capacitors:10UF-0603-6.3V-20%
- removed U3: APDS-9301, SparkFun-Sensors:APDS-9301
- added C11, C16: 1.0uF, SparkFun-Capacitors:1.0UF-0603-16V-10%
- added U$4: HN01, PWSONN6:HN01
- C10: value 0.1uF -> 10uF; device SparkFun-Capacitors:0.1UF-0603-25V-(+80/-20%) -> SparkFun-Capacitors:10UF-0603-6.3V-20%
- C12: value 1 uF -> 10uF; device Spark:C-US -> SparkFun-Capacitors:10UF-0603-6.3V-20%
- C14: value 1.0uF -> 10uF; device SparkFun-Capacitors:1.0UF-0603-16V-10% -> SparkFun-Capacitors:10UF-0603-6.3V-20%
- C15: value 10uF -> 1.0uF; device SparkFun-Capacitors:10UF-0603-6.3V-20% -> SparkFun-Capacitors:1.0UF-0603-16V-10%
- C2: device SparkFun-Capacitors:0.1UF-0603-25V-5% -> SparkFun-Capacitors:0.1UF-0603-25V-(+80/-20%)
- renumbered C5 to C3, C6 to C13
Connections:
- net 3.3V: now also C11.1, C12.1, C16.1; no longer C12.2, C7.1, C8.1, C9.1, U3.VDD
- net GND: now also C11.2, C12.2, C16.2; no longer C12.1, C7.2, C8.2, C9.2, U3.GND
- net I2C_EN: now also U$4.P$1
- net SCL: no longer U3.SCL
- net SDA: no longer U3.SDA
Other:
- note removed: "2.7V < VCC < 3.6V"
- note removed: "I2C Address Defalt 0x39 - FLOAT (0x49 - GN) (0x29 - HIGH)"
- moved on the sheet: C10, C14, C15, C2, C4
