File: Lagopus_Board/Lagopus_B.sch (EAGLE design)
At the start: 10 parts, among them J1 PTH, U1 TMP1021:1, U3 BME280

Commit message: Ordered Version 1.0 from Seeed
Lemming_SMD V1.0
Lagopus_A V1.0
Lagopus_B V1.0
Parts:
- C2: device SparkFun-Capacitors:0.1UF-25V(+80/-20%)(0603) -> SparkFun-Capacitors:0.1UF-0603-25V-(+80/-20%)
- R2: value 10K -> 10k; device SparkFun-Resistors:10KOHM-1/10W-1%(0603)0603 -> SparkFun-Resistors:10KOHM-0603-1/10W-1%
- renumbered R13 to R3, R14 to R4
Changed lines of the file:
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@@
 <part name="SUPPLY14" library="SparkFun-PowerSymbols" deviceset="3.3V" device=""/>
 <part name="U3" library="SparkFun-Sensors" deviceset="BME280" device="" value="BME280"/>
-<part name="C2" library="SparkFun-Capacitors" deviceset="0.1UF-25V(+80/-20%)(0603)" device="" value="0.1uF"/>
 <part name="U1" library="SparkFun-Sensors" deviceset="TMP102" device="1:1"/>
 <part name="GND1" library="SparkFun" deviceset="GND" device=""/>
 <part name="GND" library="SparkFun" deviceset="GND" device=""/>
-<part name="R2" library="SparkFun-Resistors" deviceset="10KOHM-1/10W-1%(0603)" device="0603" value="10K"/>
 <part name="GND4" library="SparkFun-PowerSymbols" deviceset="GND" device=""/>
 <part name="SUPPLY4" library="SparkFun-PowerSymbols" deviceset="3.3V" device=""/>
@@
 <part name="SUPPLY3" library="SparkFun-PowerSymbols" deviceset="3.3V" device=""/>
 <part name="GND5" library="SparkFun" deviceset="GND" device=""/>
-<part name="R13" library="SparkFun-Resistors" deviceset="4.7KOHM" device="-0603-1/10W-1%" value="4.7k"/>
-<part name="R14" library="SparkFun-Resistors" deviceset="4.7KOHM" device="-0603-1/10W-1%" value="4.7k"/>
+<part name="R3" library="SparkFun-Resistors" deviceset="4.7KOHM" device="-0603-1/10W-1%" value="4.7k"/>
+<part name="R4" library="SparkFun-Resistors" deviceset="4.7KOHM" device="-0603-1/10W-1%" value="4.7k"/>
 <part name="SUPPLY2" library="SparkFun-PowerSymbols" deviceset="3.3V" device=""/>
 <part name="JP2" library="SparkFun-Jumpers" deviceset="JUMPER-SMT_3_2-NC_PASTE" device="_SILK" value=""/>
 <part name="SUPPLY5" library="SparkFun-PowerSymbols" deviceset="3.3V" device=""/>
+<part name="C2" library="SparkFun-Capacitors" deviceset="0.1UF" device="-0603-25V-(+80/-20%)" value="0.1uF"/>
+<part name="R2" library="SparkFun-Resistors" deviceset="10KOHM" device="-0603-1/10W-1%" value="10k"/>
 </parts>
 <sheets>
@@
 <instance part="SUPPLY14" gate="G$1" x="0" y="78.74"/>
 <instance part="U3" gate="U1" x="27.94" y="71.12"/>
-<instance part="C2" gate="G$1" x="132.08" y="76.2" rot="MR0"/>
 <instance part="U1" gate="G$1" x="172.72" y="76.2"/>
 <instance part="GND1" gate="1" x="152.4" y="63.5"/>
 <instance part="GND" gate="1" x="195.58" y="53.34"/>
-<instance part="R2" gate="G$1" x="195.58" y="63.5" rot="R90"/>
 <instance part="GND4" gate="1" x="30.48" y="-20.32" rot="MR0"/>
 <instance part="SUPPLY4" gate="G$1" x="30.48" y="-2.54" rot="MR0"/>
@@
 <instance part="SUPPLY3" gate="G$1" x="132.08" y="88.9"/>
 <instance part="GND5" gate="1" x="132.08" y="63.5"/>
-<instance part="R13" gate="G$1" x="-12.7" y="-15.24" rot="R90"/>
-<instance part="R14" gate="G$1" x="2.54" y="-15.24" rot="R90"/>
+<instance part="R3" gate="G$1" x="-12.7" y="-15.24" rot="R90"/>
+<instance part="R4" gate="G$1" x="2.54" y="-15.24" rot="R90"/>
 <instance part="SUPPLY2" gate="G$1" x="-5.08" y="2.54"/>
 <instance part="JP2" gate="G$1" x="-5.08" y="-5.08" smashed="yes" rot="R270">
@@
 </instance>
 <instance part="SUPPLY5" gate="G$1" x="60.96" y="78.74"/>
+<instance part="C2" gate="G$1" x="132.08" y="76.2"/>
+<instance part="R2" gate="G$1" x="195.58" y="63.5" rot="R90"/>
 </instances>
 <busses>
@@
 </segment>
 <segment>
-<pinref part="R2" gate="G$1" pin="1"/>
 <pinref part="GND" gate="1" pin="GND"/>
 <wire x1="195.58" y1="55.88" x2="195.58" y2="58.42" width="0.1524" layer="91"/>
-</segment>
-<segment>
-<pinref part="C2" gate="G$1" pin="2"/>
+<pinref part="R2" gate="G$1" pin="1"/>
+</segment>
+<segment>
 <pinref part="GND5" gate="1" pin="GND"/>
 <wire x1="132.08" y1="73.66" x2="132.08" y2="66.04" width="0.1524" layer="91"/>
+<pinref part="C2" gate="G$1" pin="2"/>
 </segment>
 </net>
@@
 </segment>
 <segment>
-<pinref part="R14" gate="G$1" pin="1"/>
+<pinref part="R4" gate="G$1" pin="1"/>
 <wire x1="2.54" y1="-20.32" x2="2.54" y2="-22.86" width="0.1524" layer="91"/>
 <label x="2.54" y="-22.86" size="1.27" layer="95" rot="R270" xref="yes"/>
@@
 </segment>
 <segment>
-<pinref part="R13" gate="G$1" pin="1"/>
+<pinref part="R3" gate="G$1" pin="1"/>
 <wire x1="-12.7" y1="-22.86" x2="-12.7" y2="-20.32" width="0.1524" layer="91"/>
 <label x="-12.7" y="-22.86" size="1.27" layer="95" rot="R270" xref="yes"/>
@@
 </segment>
 <segment>
-<pinref part="C2" gate="G$1" pin="1"/>
 <pinref part="SUPPLY3" gate="G$1" pin="3.3V"/>
 <wire x1="132.08" y1="81.28" x2="132.08" y2="88.9" width="0.1524" layer="91"/>
+<pinref part="C2" gate="G$1" pin="1"/>
 </segment>
 <segment>
@@
 <pinref part="U1" gate="G$1" pin="ADD0"/>
 <wire x1="182.88" y1="71.12" x2="195.58" y2="71.12" width="0.1524" layer="91"/>
+<wire x1="195.58" y1="68.58" x2="195.58" y2="71.12" width="0.1524" layer="91"/>
 <pinref part="R2" gate="G$1" pin="2"/>
-<wire x1="195.58" y1="68.58" x2="195.58" y2="71.12" width="0.1524" layer="91"/>
 </segment>
 </net>
 <net name="N$7" class="0">
 <segment>
-<pinref part="R13" gate="G$1" pin="2"/>
+<pinref part="R3" gate="G$1" pin="2"/>
 <wire x1="-12.7" y1="-10.16" x2="-12.7" y2="-5.08" width="0.1524" layer="91"/>
 <pinref part="JP2" gate="G$1" pin="3"/>
@@
 <net name="N$8" class="0">
 <segment>
-<pinref part="R14" gate="G$1" pin="2"/>
+<pinref part="R4" gate="G$1" pin="2"/>
 <wire x1="2.54" y1="-10.16" x2="2.54" y2="-5.08" width="0.1524" layer="91"/>
 <pinref part="JP2" gate="G$1" pin="1"/>
