File: Lagopus_Board/Lagopus_A_2.brd (EAGLE design)
At the start: 88.9 x 71.2 mm, 62 parts, among them J1 PTH, J2 PTH, J7 Flash Programming, U1 MLX90614_, U10 AS72652, U2 VL53L1X, U3 AS72651, U4 4MB Flash, U5 AS72652, U6 AS72651, U7 AS72653, U8 MX25L4006E, U9 AS72653

Commit message: Lagopus v2.0 Finished
Parts:
- removed C1: 4.7uF, SparkFun-Capacitors:0603
- removed C10, C14, C18, C3, C7, C9: 10uF, SparkFun-Capacitors:0603
- removed C13, C15, C16, C6: 1.0uF, SparkFun-Capacitors:0603
- removed C17, C2, C4, C5, C8: 0.1uF, SparkFun-Capacitors:0603
- removed FRAME1: FRAME-LETTER, SparkFun-Aesthetics:CREATIVE_COMMONS
- removed GND/VCC: M021X02_NO_SILK, SparkFun-Connectors:1X02_NO_SILK@1
- removed JP1: (no value), SparkFun-Jumpers:SMT-JUMPER_3_2-NC_PASTE_SILK
- removed R1, R10, R7, R8, R9: 10k, SparkFun-Resistors:0603
- removed R12, R15, R6: 10 K, Spark:R0402_B
- removed R13, R14: 4.7k, SparkFun-Resistors:0603
- removed R16, R17: 4K7, Spark:R0402_B
- removed R18: 100K, Spark:R0402_B
- removed R19: 2.2k, SparkFun-Resistors:0603
- removed U$1, U$2, U$4, U$7, U$8: HN01, PWSONN6:HN01
- removed U10: AS72652, Qwiic_Spectral_Sensor-AS7265x:LGA20
- removed U7: AS72653, kris:AS7265X
- removed U8: MX25L4006E, kris:USON-8
- removed U9: AS72653, Qwiic_Spectral_Sensor-AS7265x:LGA20
- added C21, C31, C41, C51: 10uF, SparkFun-Capacitors:0603
- added C22, C32, C42, C52: 0.1uF, SparkFun-Capacitors:0603
- added C61: 1.0uF, SparkFun-Capacitors:0603
- added R31, R32, R41, R42, R51, R52: 10k, SparkFun-Resistors:0603
- C11: value 1.0uF -> 4.7uF
- C12: value 10uF -> 0.1uF
- JP2: value (none) -> JUMPER-SMT_3_NO_SILK; device SparkFun-Jumpers:SMT-JUMPER_2_NO_SILK -> SparkFun-Jumpers:SMT-JUMPER_3_NO_SILK
- R11: value 2.2k -> 10k
- R2: value 10 K -> 4.7k; device Spark:R0402_B -> SparkFun-Resistors:0603
- R3: value 10k -> 4.7k
- R4: value 10k -> 2.2k
- R5: value 10 K -> 2.2k; device Spark:R0402_B -> SparkFun-Resistors:0603
- U1: value MLX90614_ -> VL53L1X; device SparkFun:TO-39 -> SparkFun-Sensors:VL53L1X
- U2: value VL53L1X -> MLX90614_; device SparkFun-Sensors:VL53L1X -> SparkFun:TO-39
- U4: value 4MB Flash -> AS72652; device SparkFun-IC-Memory:SO08 -> Qwiic_Spectral_Sensor-AS7265x:LGA20
- U5: value AS72652 -> AS72653; device kris:AS7265X -> Qwiic_Spectral_Sensor-AS7265x:LGA20
- U6: value AS72651 -> 4MB Flash; device kris:AS7265X -> SparkFun-IC-Memory:SO08
- moved TP1 140.7 mm to (11.2, 40.6)
- moved J4 139.5 mm to (7.87, 40.4), turned to 180 degrees
- moved R4 117.0 mm to (13.0, 29.2), turned to 270 degrees
- moved R11 108.0 mm to (27.2, 20.3), turned to 90 degrees
- moved U3 103.8 mm to (8.89, 35.6), turned to 180 degrees
- moved U4 102.3 mm to (0.00, 35.6), turned to 180 degrees
- moved J7 91.9 mm to (12.2, 22.7), flipped to the bottom, turned to 180 degrees
- moved U1 40.2 mm to (22.9, 20.3), turned to 90 degrees
- moved C12 35.7 mm to (22.9, 28.2), turned to 0 degrees
- moved U2 29.8 mm to (-22.9, 20.3), turned to 270 degrees
- moved R2 24.6 mm to (-9.14, 16.5), turned to 90 degrees
- moved JP2 22.4 mm to (-10.4, 20.3), turned to 0 degrees
- moved R3 21.7 mm to (-11.7, 16.5)
- moved U6 20.8 mm to (12.2, 22.7), turned to 0 degrees
- moved C11 17.8 mm to (22.9, 26.2), turned to 0 degrees
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Connections:
- removed net !CS: R18.1, U$7.P$1, U5.P$6, U8.P$1
- removed net DRV1: U5.P$15
- removed net DRV2: U7.P$15
- removed net DRV3: U6.P$15
- removed net I2C_EN: JP2.2, R3.1, U$4.P$1, U5.P$8
- removed net IND1: U5.P$18
- removed net RX/SCL: U3.11
- removed net SCL_M: R17.1, U5.P$9, U6.P$9, U7.P$9
- removed net SDA_M: R16.1, U5.P$10, U6.P$10, U7.P$10
- removed net SI: U$1.P$1, U5.P$4, U8.P$5
- removed net SLV1_RESN: R12.1, U5.P$1, U7.P$2
- removed net SLV2_RESN: R15.1, U5.P$20, U6.P$2
- removed net SO: U$8.P$1, U5.P$5, U8.P$2
- removed net TX/SDA: U3.12
- net !CS_EE: now also U6.1; no longer U4.1
- net !INT: no longer GND/VCC.2, R6.1, U5.P$13
- net !RST: now also R31.1, U5.2; no longer GND/VCC.1, R4.1, R5.1, U5.P$2, U9.2
- net !RST-ADDR: now also U4.2; no longer U10.2
- net !SHUT: now also R11.1, U1.5; no longer R2.1, U2.5
- net 3.3V: now also C21.1, C22.1, C31.1, C32.1, C41.1, C42.1, C51.1, C52.1, C61.1, JP2.2, R31.2, R32.2, U1.1, U1.11, U2.3, U4.14, U4.17, U5.14, U5.17, U6.3, U6.7, U6.8; no longer C1.1, C10.1, C13.1, C14.1, C15.1, C16.1, C17.1, C18.1, C2.1, C3.1, C4.1, C5.1, C6.1, C7.1, C8.1, C9.1, JP1.2, R1.2, R12.2, R15.2, R16.2, R17.2, R18.2, R19.2, R2.2, R3.2, R6.2, U1.3, U10.14, U10.17, U2.1, U2.11, U4.3, U4.7, U4.8, U5.P$14, U5.P$17, U6.P$14, U6.P$17, U7.P$14, U7.P$17, U8.P$3, U8.P$7, U8.P$8, U9.14, U9.17
- net GND: now also C21.2, C22.2, C31.2, C32.2, C41.2, C42.2, C51.2, C52.2, C61.2, R41.1, R42.1, R51.1, R52.1, U1.12, U1.2, U1.3, U1.6, U4.16, U5.16, U6.4; no longer C1.2, C10.2, C13.2, C14.2, C15.2, C16.2, C17.2, C18.2, C2.2, C3.2, C4.2, C5.2, C6.2, C7.2, C8.2, C9.2, JP2.1, R10.1, R7.1, R8.1, R9.1, U10.16, U2.12, U2.2, U2.3, U2.6, U4.4, U5.P$16, U6.P$16, U7.P$16, U8.P$4, U9.16
- net I2C_ENB: now also R32.1; no longer R1.1
- net MISO: now also U6.2; no longer U4.2
- net MOSI: now also U6.5; no longer U4.5
- net N$10: now also R42.2, U4.5; no longer R7.2, U10.5
- net N$12: now also R51.2, U5.7; no longer R10.2, U9.7
- net N$13: now also R52.2, U5.5; no longer R9.2, U9.5
- net N$7: now also JP2.3, R2.2; no longer JP1.3, R13.2
- net N$8: now also JP2.1, R3.2; no longer JP1.1, R14.2
- net N$9: now also R41.2, U4.7; no longer R8.2, U10.7
- net SCK: now also U6.6; no longer U$2.P$1, U4.6, U5.P$3, U8.P$6
- net SCL: now also R3.1, U1.10, U2.1, U3.11; no longer R14.1, U1.1, U2.10, U5.P$11
- net SCL_S: now also R5.1, U4.9, U5.9; no longer R11.1, U10.9, U9.9
- net SDA: now also R2.1, U1.9, U2.2, U3.12; no longer R13.1, U1.2, U2.9, U5.P$12
- net SDA_S: now also R4.1, U4.10, U5.10; no longer R19.1, U10.10, U9.10
Routing:
- net SDA_S: track 0.00 -> 37.8 mm, vias 0 -> 3
- net !INT: track 39.9 -> 2.78 mm, vias 1 -> 0
- net SCL: track 67.0 -> 104.1 mm
- net I2C_EN: track 35.9 -> 0.00 mm, vias 2 -> 0
- net SCL_S: track 0.00 -> 31.5 mm, vias 0 -> 3
- net SDA: track 75.4 -> 106.3 mm
- net !CS_EE: track 0.00 -> 27.2 mm, vias 0 -> 2
- net MISO: track 0.00 -> 25.4 mm, vias 0 -> 1
- net SLV2_RESN: track 25.3 -> 0.00 mm, vias 4 -> 0
- net !CS: track 25.1 -> 0.00 mm, vias 1 -> 0
- net SI: track 22.8 -> 0.00 mm, vias 1 -> 0
- net SDA_M: track 22.4 -> 0.00 mm, vias 3 -> 0
- net SO: track 21.1 -> 0.00 mm, vias 1 -> 0
- net SCL_M: track 21.0 -> 0.00 mm, vias 1 -> 0
- net SLV1_RESN: track 19.7 -> 0.00 mm, vias 2 -> 0
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
Commit message: WSN 2 ready for quotations
Parts:
- removed J4: (no value), SparkFun-Connectors:1X02_NO_SILK
- removed J7: Flash Programming, SparkFun-Connectors:2X3_TEST_POINTS
- added J3: (no value), SparkFun-Connectors:2X6_SMD
- moved C61 12.1 mm to (19.1, 29.2), turned to 90 degrees
- moved C22 5.95 mm to (-27.4, 24.9), turned to 225 degrees
- moved TP1 5.47 mm to (16.3, 38.6)
- moved C21 5.11 mm to (-29.0, 26.4), turned to 225 degrees
- moved U6 3.30 mm to (15.2, 24.0), turned to 90 degrees
- moved C11 3.06 mm to (23.1, 29.2), turned to 90 degrees
- moved C12 2.05 mm to (21.1, 29.2), turned to 90 degrees
Connections:
- net !CS_EE: now also J3.9; no longer J7.5
- net !INT: now also J3.8; no longer J4.1
- net !RST: now also J3.10; no longer J4.2
- net 3.3V: now also J3.1, J3.11; no longer J7.2
- net GND: now also J3.12, J3.2; no longer J7.6
- net MISO: now also J3.5; no longer J7.1
- net MOSI: now also J3.6; no longer J7.4
- net SCK: now also J3.7; no longer J7.3
- net SCL: now also J3.3
- net SDA: now also J3.4
Routing:
- net !INT: track 2.78 -> 53.6 mm, vias 0 -> 2
- net !RST: track 35.2 -> 80.8 mm, vias 2 -> 3
- net SCK: track 14.6 -> 42.8 mm, vias 2 -> 3
- net MOSI: track 18.2 -> 46.4 mm, vias 2 -> 3
- net 3.3V: track 158.9 -> 182.2 mm, vias 0 -> 5
- net !CS_EE: track 27.2 -> 48.3 mm, vias 2 -> 3
- net MISO: track 25.4 -> 41.2 mm, vias 1 -> 3
- net SCL: track 104.1 -> 119.4 mm, vias 2 -> 4
- net SDA: track 106.3 -> 118.3 mm
- net I2C_ENB: track 17.3 -> 18.3 mm
- net GND: vias 24 -> 26

Commit message: Order of v2
Parts:
- U2: value MLX90614_ -> MLX90614; device SparkFun:TO-39 -> Lagopus_A_2:TO-39
- U3, U4, U5: device Qwiic_Spectral_Sensor-AS7265x:LGA20 -> Lagopus_A_2:LGA20
- U6: device SparkFun-IC-Memory:SO08 -> Lagopus_A_2:SO08
- renumbered J3 to J4
Routing:
- net GND: track 1.29 -> 5.88 mm
- net 3.3V: track 182.2 -> 184.2 mm
- net !CS_EE: track 48.3 -> 49.6 mm
- net SCL_S: track 31.5 -> 32.4 mm
- net SDA_S: track 37.6 -> 38.3 mm
