File: Lagopus_Board/Lagopus_A_2.sch (EAGLE design)
At the start: 61 parts, among them J1 PTH, J2 PTH, J7 Flash Programming, U1 MLX90614_, U10 AS72652, U2 VL53L1X, U3 AS72651, U4 4MB Flash, U5 AS72652, U6 AS72651, U7 AS72653, U8 MX25L4006E, U9 AS72653

Commit message: Lagopus v2.0 Finished
Parts:
- removed C1: 4.7uF, SparkFun-Capacitors:4.7UF0603
- removed C10, C14, C18, C3, C7, C9: 10uF, SparkFun-Capacitors:10UF-0603-6.3V-20%
- removed C13, C15, C16, C6: 1.0uF, SparkFun-Capacitors:1.0UF-0603-16V-10%
- removed C17, C2, C4, C5, C8: 0.1uF, SparkFun-Capacitors:0.1UF-0603-25V-(+80/-20%)
- removed FRAME1: FRAME-LETTER, SparkFun-Aesthetics:FRAME-LETTER
- removed GND/VCC: M021X02_NO_SILK, SparkFun-Connectors:M021X02_NO_SILK
- removed JP1: JUMPER-SMT_3_2-NC_PASTE_SILK, SparkFun-Jumpers:JUMPER-SMT_3_2-NC_PASTE_SILK
- removed R1, R10, R7, R8, R9: 10k, SparkFun-Resistors:10KOHM-0603-1/10W-1%
- removed R12, R15, R6: 10 K, Spark:R-US_
- removed R13, R14: 4.7k, SparkFun-Resistors:4.7KOHM-0603-1/10W-1%
- removed R16, R17: 4K7, Spark:R-US_
- removed R18: 100K, Spark:R-US_
- removed R19: 2.2k, SparkFun-Resistors:2.2KOHM-0603-1/10W-1%
- removed U$1, U$2, U$4, U$7, U$8: HN01, PWSONN6:HN01
- removed U10: AS72652, Qwiic_Spectral_Sensor-AS7265x:AS72652
- removed U7: AS72653, kris:AS72652
- removed U8: MX25L4006E, kris:MX25L4006E
- removed U9: AS72653, Qwiic_Spectral_Sensor-AS7265x:AS72653
- added C21, C31, C41, C51: 10uF, SparkFun-Capacitors:10UF-0603-6.3V-20%
- added C22, C32, C42, C52: 0.1uF, SparkFun-Capacitors:0.1UF-0603-25V-(+80/-20%)
- added C61: 1.0uF, SparkFun-Capacitors:1.0UF-0603-16V-10%
- added R31, R32, R41, R42, R51, R52: 10k, SparkFun-Resistors:10KOHM-0603-1/10W-1%
- C11: value 1.0uF -> 4.7uF; device SparkFun-Capacitors:1.0UF-0603-16V-10% -> SparkFun-Capacitors:4.7UF0603
- C12: value 10uF -> 0.1uF; device SparkFun-Capacitors:10UF-0603-6.3V-20% -> SparkFun-Capacitors:0.1UF-0603-25V-(+80/-20%)
- JP2: value JUMPER-SMT_2_NO_SILK -> JUMPER-SMT_3_NO_SILK; device SparkFun-Jumpers:JUMPER-SMT_2_NO_SILK -> SparkFun-Jumpers:JUMPER-SMT_3_NO_SILK
- R11: value 2.2k -> 10k; device SparkFun-Resistors:2.2KOHM-0603-1/10W-1% -> SparkFun-Resistors:10KOHM-0603-1/10W-1%
- R2: value 10 K -> 4.7k; device Spark:R-US_ -> SparkFun-Resistors:4.7KOHM-0603-1/10W-1%
- R3: value 10k -> 4.7k; device SparkFun-Resistors:10KOHM-0603-1/10W-1% -> SparkFun-Resistors:4.7KOHM-0603-1/10W-1%
- R4: value 10k -> 2.2k; device SparkFun-Resistors:10KOHM-0603-1/10W-1% -> SparkFun-Resistors:2.2KOHM-0603-1/10W-1%
- R5: value 10 K -> 2.2k; device Spark:R-US_ -> SparkFun-Resistors:2.2KOHM-0603-1/10W-1%
- U1: value MLX90614_ -> VL53L1X; device SparkFun:MLX90614_ -> SparkFun-Sensors:VL53L1XSMD
- U2: value VL53L1X -> MLX90614_; device SparkFun-Sensors:VL53L1XSMD -> SparkFun:MLX90614_
- U4: value 4MB Flash -> AS72652; device SparkFun-IC-Memory:AT25SF041 -> Qwiic_Spectral_Sensor-AS7265x:AS72652
- U5: value AS72652 -> AS72653; device kris:AS7265X -> Qwiic_Spectral_Sensor-AS7265x:AS72653
- U6: value AS72651 -> 4MB Flash; device kris:AS72652 -> SparkFun-IC-Memory:AT25SF041
Connections:
- removed net !CS: R18.1, U$7.P$1, U5.!CS_EE, U8.!CS
- removed net DRV1: U5.LED_DRV
- removed net DRV2: U7.LED_DRV
- removed net DRV3: U6.LED_DRV
- removed net I2C_EN: JP2.2, R3.1, U$4.P$1, U5.I2C_EN
- removed net IND1: U5.LED_IND
- removed net RX/SCL: U3.RX/SCL
- removed net SCL_M: R17.1, U5.!INT, U6.SCL_S, U7.SCL_S
- removed net SDA_M: R16.1, U5.NC10, U6.SDA_S, U7.SDA_S
- removed net SI: U$1.P$1, U5.MOSI, U8.SI
- removed net SLV1_RESN: R12.1, U5.SDA_M, U7.!RST
- removed net SLV2_RESN: R15.1, U5.SCL_M, U6.!RST
- removed net SO: U$8.P$1, U5.MISO, U8.SO
- removed net TX/SDA: U3.TX/SDA
- net !CS_EE: now also U6.!CS; no longer U4.!CS
- net !INT: no longer GND/VCC.2, R6.1, U5.ADO
- net !RST: now also R31.1; no longer GND/VCC.1, R4.1, R5.1, U9.!RST
- net !RST-ADDR: now also U4.!RST; no longer U10.!RST
- net !SHUT: now also R11.1, U1.!SHUT; no longer R2.1, U2.!SHUT
- net 3.3V: now also C21.1, C22.1, C31.1, C32.1, C41.1, C42.1, C51.1, C52.1, C61.1, JP2.2, R31.2, R32.2, U1.VCC, U2.VDD, U4.VDD, U5.VDD, U6.!HOLD(D3), U6.!WP(D2), U6.VCC; no longer C1.1, C10.1, C13.1, C14.1, C15.1, C16.1, C17.1, C18.1, C2.1, C3.1, C4.1, C5.1, C6.1, C7.1, C8.1, C9.1, JP1.2, R1.2, R12.2, R15.2, R16.2, R17.2, R18.2, R19.2, R2.2, R3.2, R6.2, U1.VDD, U10.VDD, U2.VCC, U4.!HOLD(D3), U4.!WP(D2), U4.VCC, U5.VDD1, U5.VDD2, U6.VDD1, U6.VDD2, U7.VDD1, U7.VDD2, U8.!HOLD, U8.!WP, U8.VCC, U9.VDD
- net GND: now also C21.2, C22.2, C31.2, C32.2, C41.2, C42.2, C51.2, C52.2, C61.2, R41.1, R42.1, R51.1, R52.1, U1.GND, U2.VSS; no longer C1.2, C10.2, C13.2, C14.2, C15.2, C16.2, C17.2, C18.2, C2.2, C3.2, C4.2, C5.2, C6.2, C7.2, C8.2, C9.2, JP2.1, R10.1, R7.1, R8.1, R9.1, U1.VSS, U10.GND, U2.GND, U7.GND, U8.GND, U9.GND
- net I2C_ENB: now also R32.1; no longer R1.1
- net MISO: now also U6.SO(D1); no longer U4.SO(D1)
- net MOSI: now also U6.SI(D0); no longer U4.SI(D0)
- net N$10: now also R42.2, U4.MISO; no longer R7.2, U10.MISO
- net N$12: now also R51.2, U5.!CS_SD; no longer R10.2, U9.!CS_SD
- net N$13: now also R52.2, U5.MISO; no longer R9.2, U9.MISO
- net N$7: now also JP2.3, R2.2; no longer JP1.3, R13.2
- net N$8: now also JP2.1, R3.2; no longer JP1.1, R14.2
- net N$9: now also R41.2, U4.!CS_SD; no longer R8.2, U10.!CS_SD
- net SCK: now also U6.SCK; no longer U$2.P$1, U4.SCK, U5.SCK, U8.SCLK
- net SCL: now also R3.1, U1.SCL, U2.SCL/VZ, U3.RX/SCL; no longer R14.1, U1.SCL/VZ, U2.SCL, U5.RX/SCL_S
- net SCL_S: now also R5.1, U4.SCL_S, U5.SCL_S; no longer R11.1, U10.SCL_S, U9.SCL_S
- net SDA: now also R2.1, U1.SDA, U2.PWM/SDA, U3.TX/SDA; no longer R13.1, U1.PWM/SDA, U2.SDA, U5.TX/SDA_S
- net SDA_S: now also R4.1, U4.SDA_S, U5.SDA_S; no longer R19.1, U10.SDA_S, U9.SDA_S
Other:
- note added: "MLX90614 IR-Temp"
- note removed: "Clear jumper JP9 to remove pull-up from INT"
- note removed: "Nathan Seidle"
- note removed: "Open(Default) - I2C Operation Closed - Serial Operation"
- note removed: "VCC: 2.3V-3.5V"
- note removed: "X10"
- moved on the sheet: C11, C12, J1, J2, J4, J7, R11, R2, R3, R4, R5, TP1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

Commit message: WSN 2 ready for quotations
Parts:
- removed J4: (no value), SparkFun-Connectors:CONN_021X02_NO_SILK
- removed J7: Flash Programming, SparkFun-Connectors:AVR_SPI_PROG_3X2TESTPOINTS
- added J3: (no value), SparkFun-Connectors:CONN_06X2SMD_FEMALE
Connections:
- net !CS_EE: now also J3.9; no longer J7.5
- net !INT: now also J3.8; no longer J4.1
- net !RST: now also J3.10; no longer J4.2
- net 3.3V: now also J3.1, J3.11; no longer J7.2
- net GND: now also J3.12, J3.2; no longer J7.6
- net MISO: now also J3.5; no longer J7.1
- net MOSI: now also J3.6; no longer J7.4
- net SCK: now also J3.7; no longer J7.3
- net SCL: now also J3.3
- net SDA: now also J3.4
Other:
- moved on the sheet: C61, U6

Commit message: Order of v2
Parts:
- U2: value MLX90614_ -> MLX90614; device SparkFun:MLX90614_ -> Lagopus_A_2:MLX90614
- U3: device Qwiic_Spectral_Sensor-AS7265x:AS72651 -> Lagopus_A_2:AS72651
- U4: device Qwiic_Spectral_Sensor-AS7265x:AS72652 -> Lagopus_A_2:AS72652
- U5: device Qwiic_Spectral_Sensor-AS7265x:AS72653 -> Lagopus_A_2:AS72653
- U6: device SparkFun-IC-Memory:AT25SF041 -> Lagopus_A_2:AT25SF041
- renumbered J3 to J4
Other:
- moved on the sheet: U2
