File: Lagopus_Board/Lagopus_B_2.sch (EAGLE design)
At the start: 10 parts, among them J1 PTH, U1 SHT31-DIS-F, U3 BME280, U4 TMP117

Commit message: Order of v2
Parts:
- U1: device microbuilder:SHT3X -> Lagopus_B_2:SHT3X
- U4: device SparkFun-Sensors:TMP117 -> Lagopus_B_2:TMP117
Other:
- moved on the sheet: U4
Changed lines of the file:
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@@
 <part name="GND6" library="SparkFun" deviceset="GND" device=""/>
 <part name="C3" library="SparkFun-Capacitors" deviceset="0.1UF" device="-0603-25V-(+80/-20%)" value="0.1uF"/>
-<part name="U4" library="SparkFun-Sensors" deviceset="TMP117" device=""/>
-<part name="U1" library="microbuilder" deviceset="SHT3X" device="" value="SHT31-DIS-F"/>
+<part name="U4" library="Lagopus_B_2" deviceset="TMP117" device=""/>
+<part name="U1" library="Lagopus_B_2" deviceset="SHT3X" device="" value="SHT31-DIS-F"/>
 <part name="GND8" library="SparkFun" deviceset="GND" device=""/>
 <part name="C4" library="SparkFun-Capacitors" deviceset="10UF" device="-0603-6.3V-20%" value="10uF"/>
