File: Lagopus_Board/Lagopus_A_3.sch (EAGLE design)
At the start: 29 parts, among them IC1 VEML7700, J1 PTH, J2 PTH, Q2 BSS138, U1 VL53L1X, U2 LAGOPUS_A_2_MLX90614, U3 LSM9DS1, X1 AS7341

Commit message: Merry Christmas
Parts:
- removed J2: PTH, SparkX:I2C_STANDARD_NO_SILK
- removed R1: 10K, microbuilder:RESISTOR_4PACK
- removed U$8: 1.8V/100mA, SparkFun-IC-Power:V_REG_SP6214-1.8V
- removed U2: LAGOPUS_A_2_MLX90614, Lagopus_A_3:LAGOPUS_A_2_MLX90614
- added C13: 10uF, SparkFun-Capacitors:10UF-0603-6.3V-20%
- added C14: 0.1uF, SparkFun-Capacitors:0.1UF-0603-25V-(+80/-20%)
- added IC2: MIC5247-1.8YM5-TR, MIC5247-1.8YM5-TR:MIC5247-1.8YM5-TR
- added IC3: MLX90614ESF-BAA-000-TU, MLX90614ESF-BAA-000-TU:MLX90614ESF-BAA-000-TU
- added RN1, RN2: CAY16-1002F4LF, CAY16-1002F4LF:CAY16-1002F4LF
- added U4: SPARKFUN-SENSORS_VCNL4040, Lagopus_A_3:SPARKFUN-SENSORS_VCNL4040
- C11: value 4.7uF -> 10uF; device SparkFun-Capacitors:4.7UF0603 -> SparkFun-Capacitors:10UF-0603-6.3V-20%
Connections:
- new net N$10: RN1.8, U3.SDO_A/G
- new net N$11: RN1.5, U3.CS_M
- new net N$12: U4.CATHODE_LED, U4.CATHODE_SEN
- new net N$4: RN1.7, U3.SDO_M
- new net N$9: RN1.6, U3.CS_A/G
- net 1.8V: now also IC2.OUT, RN2.1, RN2.3; no longer R1G$2.1, R1G$4.1, U$8.OUT
- net 3.3V: now also C13.1, C14.1, IC2.EN, IC2.IN, IC3.VDD, RN1.1, RN1.2, RN1.3, RN1.4, U4.ANODE, U4.VDD; no longer J2.VCC, U$8.EN, U$8.IN, U2.VDD, U3.CS_A/G, U3.CS_M, U3.SDO_A/G, U3.SDO_M
- net GND: now also C13.2, C14.2, IC2.GND, IC3.VSS, U4.GND; no longer J2.GND, U$8.GND, U2.VSS
- net N$1: now also RN2.2; no longer R1G$3.1
- net N$2: now also RN2.4; no longer R1G$1.1
- net SCL: now also IC3.SCL/VZ, RN2.8, U4.SCL; no longer J2.SCL, R1G$1.2, U2.SCL/VZ
- net SCL_2V: now also RN2.7; no longer R1G$2.2
- net SDA: now also IC3.PWM/SDA, RN2.6, U4.SDA; no longer J2.SDA, R1G$3.2, U2.PWM/SDA
- net SDA_2V: now also RN2.5; no longer R1G$4.2
Other:
- note added: "7-bit unshifted I2C address: 0x60"
- note added: "VCNL4040 IR Proximity Sensor"
- moved on the sheet: C11, C3, C4, C5, C6, C7, C8, C9, JP1, Q2G$1, Q2G$2, U3

Commit message: Lagopus 3.0 order
Parts:
- removed C3, C7: 10uF, SparkFun-Capacitors:10UF-0603-6.3V-20%
- removed C4, C5, C6: 0.1uF, SparkFun-Capacitors:0.1UF-0603-25V-(+80/-20%)
- removed IC2: MIC5247-1.8YM5-TR, MIC5247-1.8YM5-TR:MIC5247-1.8YM5-TR
- removed RN1: CAY16-1002F4LF, CAY16-1002F4LF:CAY16-1002F4LF
- removed U3: LSM9DS1, SparkFun-Sensors:LSM9DS1
- added C15, C17: 0.1uF, SparkFun-Capacitors:0.1UF-0603-25V-(+80/-20%)
- added C16: 10uF, SparkFun-Capacitors:10UF-0603-6.3V-20%
- added R1: 4.7k, SparkFun-Resistors:4.7KOHM-0603-1/10W-1%
- added U$21: MPU-9250_ICM20948, adafruit_sensor:MPU-9250_ICM20948
- added U2: MIC5225-1.8V, microbuilder:VREG_SOT23-5
Connections:
- removed net N$10: RN1.8, U3.SDO_A/G
- removed net N$11: RN1.5, U3.CS_M
- removed net N$3: C4.1, U3.C1
- removed net N$4: RN1.7, U3.SDO_M
- removed net N$5: C7.1, U3.CAP
- removed net N$9: RN1.6, U3.CS_A/G
- new net AUX_SCL: U$21.AUX_CL
- new net AUX_SDA: U$21.AUX_DA
- new net FSYNC: U$21.FSYNC
- new net INT_1.8V: U$21.INT
- new net N$13: C15.1, U$21.REGOUT
- new net N$14: R1.1, U$21.!CS, U$21.AD0/SDO
- net 1.8V: now also C16.1, C17.1, Q21.G, Q22.G, R1.2, U$21.VDD, U$21.VDDIO, U2.OUT; no longer IC2.OUT, Q2G$1.G, Q2G$2.G
- net 3.3V: now also U2.EN, U2.IN; no longer C3.1, C5.1, C6.1, IC2.EN, IC2.IN, RN1.1, RN1.2, RN1.3, RN1.4, U3.VDD, U3.VDDIO
- net GND: now also C15.2, C16.2, C17.2, U$21.GND, U2.GND; no longer C3.2, C4.2, C5.2, C6.2, C7.2, IC2.GND, U3.GND, U3.RES
- net SCL: now also Q21.D; no longer Q2G$1.D, U3.SCL/SPC
- net SCL_2V: now also Q21.S, U$21.SCL/SCLK; no longer Q2G$1.S
- net SDA: now also Q22.D; no longer Q2G$2.D, U3.SDA/SDI/SDO
- net SDA_2V: now also Q22.S, U$21.SDA/SDI; no longer Q2G$2.S
Other:
- note added: "9DoF ICM-20948"
- note added: "AS7341"
- note added: "I2C address 0x69"
- note removed: "0x1E*"
- note removed: "0x6B*"
- note removed: "AG Addr."
- note removed: "LSM9DS1 Magnetometer, Accelerometer and Gyro"
- note removed: "M Addr."
- moved on the sheet: C8
