File: Lagopus_Board/Lagopus_A_3.brd (EAGLE design)
At the start: 88.9 x 71.2 mm, 31 parts, among them IC1 VEML7700, J1 PTH, J2 PTH, Q2 BSS138, U1 VL53L1X, U2 LAGOPUS_A_2_MLX90614, U3 LSM9DS1, X1 AS7341

Commit message: Merry Christmas
Parts:
- removed J2: PTH, SparkX:1X04_NO_SILK
- removed R1: 10K, microbuilder:RESPACK_4X0603
- removed U$8: 1.8V/100mA, SparkFun-IC-Power:SC70
- removed U2: LAGOPUS_A_2_MLX90614, Lagopus_A_3:LAGOPUS_A_2_TO-39
- added C13: 10uF, SparkFun-Capacitors:0603
- added C14: 0.1uF, SparkFun-Capacitors:0603
- added IC2: MIC5247-1.8YM5-TR, MIC5247-1.8YM5-TR:SOT95P280X145-5N
- added IC3: MLX90614ESF-BAA-000-TU, MLX90614ESF-BAA-000-TU:MLX90614ESFBAA000TU
- added RN1, RN2: CAY16-1002F4LF, CAY16-1002F4LF:CAY-16-F4
- added U4: SPARKFUN-SENSORS_VCNL4040, Lagopus_A_3:SPARKFUN-SENSORS_SPARKX_VCNL4040
- C11: value 4.7uF -> 10uF
- moved C12 63.1 mm to (-32.8, 3.56), turned to 90 degrees
- moved R11 60.2 mm to (-31.0, 3.56), turned to 270 degrees
- moved U$5 56.6 mm to (30.5, -12.7)
- moved C9 54.7 mm to (-30.0, -5.08), turned to 90 degrees
- moved C10 53.6 mm to (-31.8, -5.08), turned to 90 degrees
- moved C8 53.4 mm to (-23.9, -13.5)
- moved C11 52.3 mm to (-22.1, 3.56), turned to 270 degrees
- moved U1 52.0 mm to (-26.4, 3.56), turned to 0 degrees
- moved Q2 49.0 mm to (-27.9, -8.38), turned to 90 degrees
- moved X1 46.9 mm to (-26.4, -4.83), turned to 90 degrees
- moved JP1 46.4 mm to (-23.9, -10.7), flipped to the bottom, turned to 270 degrees
- moved C21 45.2 mm to (16.3, 27.7), turned to 90 degrees
- moved C22 43.7 mm to (16.3, 23.6), turned to 270 degrees
- moved U$2 17.7 mm to (23.4, 9.36)
- moved C3 17.1 mm to (-26.7, 12.7)
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Connections:
- new net N$10: RN1.8, U3.5
- new net N$11: RN1.5, U3.8
- new net N$12: U4.2, U4.5
- new net N$4: RN1.7, U3.6
- new net N$9: RN1.6, U3.7
- net 1.8V: now also IC2.5, RN2.1, RN2.3; no longer R1.2, R1.4, U$8.5
- net 3.3V: now also C13.1, C14.1, IC2.1, IC2.3, IC3.3, RN1.1, RN1.2, RN1.3, RN1.4, U4.3, U4.4; no longer J2.2, U$8.1, U$8.3, U2.3, U3.5, U3.6, U3.7, U3.8
- net GND: now also C13.2, C14.2, IC2.2, IC3.4, U4.1; no longer J2.1, U$8.2, U2.4
- net N$1: now also RN2.2; no longer R1.3
- net N$2: now also RN2.4; no longer R1.1
- net SCL: now also IC3.1, RN2.8, U4.8; no longer J2.4, R1.8, U2.1
- net SCL_2V: now also RN2.7; no longer R1.7
- net SDA: now also IC3.2, RN2.6, U4.7; no longer J2.3, R1.6, U2.2
- net SDA_2V: now also RN2.5; no longer R1.5
Routing:
- net 3.3V: track 34.0 -> 226.2 mm, vias 0 -> 10
- net SCL: track 19.0 -> 171.3 mm, vias 0 -> 6
- net SDA: track 16.9 -> 164.7 mm, vias 0 -> 15
- net 1.8V: track 0.00 -> 21.7 mm
- net GND: track 1.29 -> 15.1 mm, vias 7 -> 19
- net SDA_2V: track 0.00 -> 12.7 mm, vias 0 -> 3
- net SCL_2V: track 0.00 -> 6.76 mm, vias 0 -> 2
- net N$2: track 0.00 -> 3.68 mm, vias 0 -> 1
- net N$1: track 0.00 -> 3.67 mm, vias 0 -> 1
- net N$12: track 0.00 -> 3.06 mm
- net N$10: track 0.00 -> 3.01 mm
- net N$3: track 0.00 -> 1.92 mm
- net N$4: track 0.00 -> 1.86 mm
- net N$11: track 0.00 -> 1.82 mm
- net N$5: track 0.00 -> 1.75 mm
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
Commit message: Lagopus 3.0 order
Parts:
- removed C3, C7: 10uF, SparkFun-Capacitors:0603
- removed C4, C5, C6: 0.1uF, SparkFun-Capacitors:0603
- removed IC2: MIC5247-1.8YM5-TR, MIC5247-1.8YM5-TR:SOT95P280X145-5N
- removed RN1: CAY16-1002F4LF, CAY16-1002F4LF:CAY-16-F4
- removed U3: LSM9DS1, SparkFun-Sensors:LGA24-8X4
- added C15, C17: 0.1uF, SparkFun-Capacitors:0603
- added C16: 10uF, SparkFun-Capacitors:0603
- added R1: 4.7k, SparkFun-Resistors:0603
- added U$21: MPU-9250_ICM20948, adafruit_sensor:QFN24_3MM_NOEP
- added U2: MIC5225-1.8V, microbuilder:SOT23-5
- moved C10 2.30 mm to (-31.5, -2.79)
- moved C13 2.30 mm to (-31.8, 1.27)
- moved C14 2.30 mm to (-30.0, 1.27)
- moved C9 2.30 mm to (-29.7, -2.79)
- moved U4 2.30 mm to (-26.2, 1.27)
- moved C11 2.30 mm to (-21.8, 5.84)
- moved C12 2.30 mm to (-32.5, 5.84)
- moved R11 2.30 mm to (-30.7, 5.84)
- moved U1 2.30 mm to (-26.2, 5.84)
- moved X1 2.30 mm to (-26.2, -2.54)
Connections:
- removed net N$10: RN1.8, U3.5
- removed net N$11: RN1.5, U3.8
- removed net N$3: C4.1, U3.24
- removed net N$4: RN1.7, U3.6
- removed net N$5: C7.1, U3.21
- removed net N$9: RN1.6, U3.7
- new net AUX_SCL: U$21.7
- new net AUX_SDA: U$21.21
- new net FSYNC: U$21.11
- new net INT_1.8V: U$21.12
- new net N$13: C15.1, U$21.10
- new net N$14: R1.1, U$21.22, U$21.9
- net 1.8V: now also C16.1, C17.1, R1.2, U$21.13, U$21.8, U2.5; no longer IC2.5
- net 3.3V: now also U2.1, U2.3; no longer C3.1, C5.1, C6.1, IC2.1, IC2.3, RN1.1, RN1.2, RN1.3, RN1.4, U3.1, U3.22, U3.23, U3.3
- net GND: now also C15.2, C16.2, C17.2, U$21.18, U$21.20, U2.2; no longer C3.2, C4.2, C5.2, C6.2, C7.2, IC2.2, U3.14, U3.15, U3.16, U3.17, U3.18, U3.19, U3.20
- net SCL: no longer U3.2
- net SCL_2V: now also U$21.23
- net SDA: no longer U3.4
- net SDA_2V: now also U$21.24
Routing:
- net 3.3V: track 226.2 -> 183.8 mm, vias 10 -> 8
- net 1.8V: track 21.7 -> 43.2 mm, vias 0 -> 2
- net SDA: track 164.7 -> 143.4 mm, vias 15 -> 11
- net SCL: track 171.3 -> 154.5 mm, vias 6 -> 3
- net N$14: track 0.00 -> 10.7 mm, vias 0 -> 2
- net GND: track 15.1 -> 5.65 mm, vias 19 -> 18
- net SCL_2V: track 6.76 -> 14.8 mm
- net SDA_2V: track 12.7 -> 19.6 mm, vias 3 -> 4
- net N$13: track 0.00 -> 3.58 mm
- net N$10: track 3.01 -> 0.00 mm
- net N$3: track 1.92 -> 0.00 mm
- net N$4: track 1.86 -> 0.00 mm
- net N$11: track 1.82 -> 0.00 mm
- net N$5: track 1.75 -> 0.00 mm
- net N$9: track 1.71 -> 0.00 mm
Other:
- outline, holes or cut-outs redrawn

Commit message: Lagopus 3 mm.
Other:
- outline, holes or cut-outs redrawn
Changed lines of the file:
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@@
 <layer number="23" name="tOrigins" color="15" fill="1" visible="yes" active="yes"/>
 <layer number="24" name="bOrigins" color="15" fill="1" visible="yes" active="yes"/>
-<layer number="25" name="tNames" color="7" fill="1" visible="no" active="yes"/>
+<layer number="25" name="tNames" color="7" fill="1" visible="yes" active="yes"/>
 <layer number="26" name="bNames" color="7" fill="1" visible="yes" active="yes"/>
-<layer number="27" name="tValues" color="7" fill="1" visible="no" active="yes"/>
+<layer number="27" name="tValues" color="7" fill="1" visible="yes" active="yes"/>
 <layer number="28" name="bValues" color="7" fill="1" visible="yes" active="yes"/>
 <layer number="29" name="tStop" color="7" fill="3" visible="yes" active="yes"/>
@@
 <wire x1="-35.56" y1="26.7284" x2="-37.7517" y2="23.5276" width="0" layer="20"/>
 <wire x1="-37.7517" y1="23.5276" x2="-37.2513" y2="-24.2546" width="0" layer="20" curve="64.9999"/>
+<wire x1="-12.7" y1="19.05" x2="-12.7" y2="-26.67" width="0.3048" layer="22" style="shortdash"/>
+<wire x1="-2.54" y1="-4.064" x2="4.064" y2="2.54" width="4.064" layer="46"/>
 </plain>
 <attributes>
