File: Lemming_SMD/Lemming_SMD_2_2.brd (EAGLE design)
At the start: 73.7 x 50.8 mm, 51 parts, among them IC1 ISO1540, IC2 ISO1540, IC3 ISO1540, Q1 2STF2360, Q10 SS8050, Q2 SS8050, Q3 2STF2360, Q4 SS8050, Q5 2STF2360, Q6 SS8050, Q7 2STF2360, Q8 SS8050, Q9 2STF2360, U3 BME280, X1 LAGOPUS, X2 1-WIRE, X3 SDI-12, X4 MB-7389, X5 1-WIRE, X6 SDI-12, X9 I2C - GPS

Commit message: WSN 2 ready for quotations
Parts:
- removed IRIDIUM: IRIDIUM, con-molex:22-23-2051
- added X10: 2059-303/998-403, con-wago_2059:P-2059-303/998-403
- added X7, X8: 2059-302/998-403, con-wago_2059:P-2059-302/998-403
- C1: value 0.1uF -> 10uF
- R1, R10, R13, R4, R7: value 10k -> 4.7k
- R11, R14, R2, R5, R8: value 1k -> 4.7k
- R12, R15, R16, R3, R6, R9: value 2.2k -> 4.7k
- X1: value LAGOPUS -> 2059-303/998-403; device con-molex:22-23-2041 -> con-wago_2059:P-2059-303/998-403
- X2: value 1-WIRE -> 2059-303/998-403; device con-molex:22-23-2031 -> con-wago_2059:P-2059-303/998-403
- X3: value SDI-12 -> 2059-303/998-403; device con-molex:22-23-2031 -> con-wago_2059:P-2059-303/998-403
- X4: value MB-7389 -> 2059-303/998-403; device con-molex:22-23-2031 -> con-wago_2059:P-2059-303/998-403
- X5: value 1-WIRE -> 2059-302/998-403; device con-molex:22-23-2031 -> con-wago_2059:P-2059-302/998-403
- X6: value SDI-12 -> 2059-302/998-403; device con-molex:22-23-2031 -> con-wago_2059:P-2059-302/998-403
- X9: value I2C - GPS -> 2059-302/998-403; device con-molex:22-23-2041 -> con-wago_2059:P-2059-302/998-403
- moved X9 50.3 mm to (50.8, 39.1), turned to 0 degrees
- moved X1 44.1 mm to (67.5, 4.50), turned to 270 degrees
- moved X4 31.8 mm to (37.5, 4.50), turned to 270 degrees
- moved X5 22.6 mm to (29.0, 4.50), turned to 270 degrees
- moved X6 19.7 mm to (23.0, 4.50), turned to 270 degrees
- moved X3 14.1 mm to (47.5, 4.50), turned to 270 degrees
- moved X2 3.76 mm to (57.5, 4.50), turned to 270 degrees
- moved R19 1.52 mm to (47.6, 20.7)
- moved R20 1.52 mm to (50.2, 20.7)
- moved U3 1.52 mm to (53.3, 20.7)
- moved C2 1.52 mm to (53.3, 23.9)
- moved JP2 1.52 mm to (48.9, 23.9)
Connections:
- net 1RX: now also X1.L2.1, X1.L2.2; no longer X4.2
- net 2RX: now also X9.L1.1, X9.L1.2; no longer IRIDIUM.1
- net 2TX: now also X9.L2.1, X9.L2.2; no longer IRIDIUM.2
- net 3.3V_D2: now also X6.L2.1, X6.L2.2; no longer X1.4
- net 3.3V_D3: now also X8.L2.1, X8.L2.2; no longer X9.4
- net 5V_D1: now also X1.L3.1, X1.L3.2; no longer X4.3
- net 5V_D5: now also X2.L3.1, X2.L3.2; no longer X2.3, X5.3
- net 5V_D7: now also X3.L3.1, X3.L3.2, X4.L3.1, X4.L3.2; no longer X3.3, X6.3
- net BATTERY: now also X10.L2.1, X10.L2.2; no longer IRIDIUM.4
- net D4: now also X10.L1.1, X10.L1.2; no longer IRIDIUM.3
- net D6: now also X2.L2.1, X2.L2.2; no longer X2.2, X5.2
- net D8: now also X3.L2.1, X3.L2.2, X4.L2.1, X4.L2.2; no longer X3.2, X6.2
- net GND: now also X1.L1.1, X1.L1.2, X10.L3.1, X10.L3.2, X2.L1.1, X2.L1.2, X3.L1.1, X3.L1.2, X4.L1.1, X4.L1.2, X5.L1.1, X5.L1.2, X7.L1.1, X7.L1.2; no longer IRIDIUM.5, X1.1, X2.1, X3.1, X4.1, X5.1, X6.1, X9.1
- net SCL2: now also X5.L2.1, X5.L2.2; no longer X1.2
- net SCL3: now also X7.L2.1, X7.L2.2; no longer X9.2
- net SDA2: now also X6.L1.1, X6.L1.2; no longer X1.3
- net SDA3: now also X8.L1.1, X8.L1.2; no longer X9.3
Routing:
- net SCL3: track 10.6 -> 21.6 mm, vias 1 -> 2
- net SCL2: track 12.1 -> 20.9 mm, vias 1 -> 2
- net 2RX: track 5.98 -> 13.4 mm
- net 5V_D7: track 66.4 -> 73.7 mm, vias 0 -> 2
- net SDA2: track 8.98 -> 16.3 mm
- net D8: track 94.5 -> 100.6 mm, vias 2 -> 4
- net 3.3V_D3: track 57.2 -> 63.1 mm, vias 2 -> 3
- net BATTERY: track 15.8 -> 21.1 mm, vias 0 -> 1
- net SDA3: track 8.46 -> 13.7 mm
- net 3.3V_D2: track 92.1 -> 95.9 mm
- net 1RX: track 69.1 -> 72.8 mm
- net 5V_D1: track 70.5 -> 73.8 mm
- net 2TX: track 9.94 -> 13.2 mm
- net D6: track 104.5 -> 101.7 mm
- net SCL1: track 41.6 -> 39.2 mm
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Other:
- outline, holes or cut-outs redrawn
- board text added: "1RX"
- board text added: "X12"
- board text added: "X24"

Commit message: Order of v2
Parts:
- moved U$3 2.92 mm to (59.0, 28.8)
Routing:
- net GND: vias 12 -> 15
Changed lines of the file:
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@@
 <setting verticaltext="up"/>
 </settings>
-<grid distance="0.5" unitdist="mm" unit="mm" style="dots" multiple="1" display="yes" altdistance="0.0125" altunitdist="inch" altunit="inch"/>
+<grid distance="0.01" unitdist="inch" unit="inch" style="dots" multiple="1" display="yes" altdistance="0.0125" altunitdist="inch" altunit="inch"/>
 <layers>
 <layer number="1" name="Top" color="4" fill="1" visible="yes" active="yes"/>
@@
 <wire x1="47.244" y1="50.8" x2="0" y2="50.8" width="0" layer="20"/>
 <wire x1="0" y1="50.8" x2="0" y2="11.43" width="0" layer="20"/>
-<text x="71.755" y="17.145" size="1.4224" layer="25" font="vector" rot="R90">(C) 2018
+<text x="73.255" y="18.645" size="1.4224" layer="25" font="vector" rot="R90">(C) 2018
 john.hulth@geo.uio.no</text>
 <text x="41.275" y="48.26" size="1.778" layer="26" font="vector" rot="MR270">Lemming SMD V2.2</text>
@@
 <text x="67.5" y="9" size="0.8128" layer="25" rot="R270" align="center-right">1RX</text>
 <text x="70.5" y="9" size="0.8128" layer="25" rot="R270" align="center-right">GND</text>
-<text x="55.626" y="40.386" size="0.8128" layer="25" rot="R180" align="center">2RX</text>
-<text x="55.626" y="37.846" size="0.8128" layer="25" rot="R180" align="center">2TX</text>
-<text x="55.626" y="35.306" size="0.8128" layer="25" rot="R180" align="center">D4</text>
-<text x="55.626" y="30.226" size="0.8128" layer="25" rot="R180" align="center">GND</text>
-<text x="55.626" y="32.766" size="0.8128" layer="25" rot="R180" align="center">BAT</text>
+<text x="56" y="40.6" size="0.8128" layer="25" align="center-left">2RX</text>
+<text x="56" y="37.6" size="0.8128" layer="25" align="center-left">2TX</text>
+<text x="56" y="34.3" size="0.8128" layer="25" align="center-left">D4</text>
+<text x="56" y="28.274" size="0.8128" layer="25" align="center-left">GND</text>
+<text x="56" y="31.234" size="0.8128" layer="25" align="center-left">BAT</text>
 <dimension x1="0" y1="0" x2="73.66" y2="0" x3="36.83" y3="-6.985" textsize="1.778" layer="48"/>
 <text x="45.466" y="47.244" size="0.8128" layer="25" rot="R90">X12</text>
@@
 <attribute name="VALUE" x="56.515" y="22.098" size="1.27" layer="25" rot="R90" align="center"/>
 </element>
-<element name="U$3" library="UIO-John" package="UIO-LOGO-BL" value="" x="56.515" y="27.305" smashed="yes"/>
+<element name="U$3" library="UIO-John" package="UIO-LOGO-BL" value="" x="59.015" y="28.805" smashed="yes"/>
 <element name="IC1" library="texas" library_urn="urn:adsk.eagle:library:387" package="SO-08" package3d_urn="urn:adsk.eagle:package:7566865/2" value="ISO1540" x="28.575" y="17.78" smashed="yes" rot="R180">
 <attribute name="MF" value="" x="28.575" y="17.78" size="1.778" layer="27" rot="R180" display="off"/>
@@
 <contactref element="X4" pad="L1.1"/>
 <via x="36" y="8.775" extent="1-16" drill="0.4"/>
+<via x="10.033" y="3.302" extent="1-16" drill="0.4"/>
+<via x="22.987" y="3.302" extent="1-16" drill="0.4"/>
+<via x="9.525" y="36.576" extent="1-16" drill="0.4"/>
 </signal>
 <signal name="1RX">
