File: Lemming_SMD/Lemming_SMD_2_2.sch (EAGLE design)
At the start: 50 parts, among them IC1 ISO1540, IC2 ISO1540, IC3 ISO1540, Q1 2STF2360, Q10 SS8050, Q2 SS8050, Q3 2STF2360, Q4 SS8050, Q5 2STF2360, Q6 SS8050, Q7 2STF2360, Q8 SS8050, Q9 2STF2360, U3 BME280, X1 LAGOPUS, X2 1-WIRE, X3 SDI-12, X4 MB-7389, X5 1-WIRE, X6 SDI-12, X9 I2C - GPS

Commit message: WSN 2 ready for quotations
Parts:
- removed IRIDIUM: IRIDIUM, con-molex:22-23-2051
- added X10: 2059-303/998-403, con-wago_2059:2059-303/998-403
- added X7, X8: 2059-302/998-403, con-wago_2059:2059-302/998-403
- C1: value 0.1uF -> 10uF; device SparkFun-Capacitors:0.1UF-0603-25V-(+80/-20%) -> SparkFun-Capacitors:10UF-0603-6.3V-20%
- R1, R10, R13, R4, R7: value 10k -> 4.7k
- R11, R14, R2, R5, R8: value 1k -> 4.7k
- R12, R15, R16, R3, R6, R9: value 2.2k -> 4.7k
- X1: value LAGOPUS -> 2059-303/998-403; device con-molex:22-23-2041 -> con-wago_2059:2059-303/998-403
- X2: value 1-WIRE -> 2059-303/998-403; device con-molex:22-23-2031 -> con-wago_2059:2059-303/998-403
- X3: value SDI-12 -> 2059-303/998-403; device con-molex:22-23-2031 -> con-wago_2059:2059-303/998-403
- X4: value MB-7389 -> 2059-303/998-403; device con-molex:22-23-2031 -> con-wago_2059:2059-303/998-403
- X5: value 1-WIRE -> 2059-302/998-403; device con-molex:22-23-2031 -> con-wago_2059:2059-302/998-403
- X6: value SDI-12 -> 2059-302/998-403; device con-molex:22-23-2031 -> con-wago_2059:2059-302/998-403
- X9: value I2C - GPS -> 2059-302/998-403; device con-molex:22-23-2041 -> con-wago_2059:2059-302/998-403
Connections:
- net 1RX: now also X1.P2.1, X1.P2.2; no longer X4-2.S
- net 2RX: now also X9.P1.1, X9.P1.2; no longer IRIDIUM-1.S
- net 2TX: now also X9.P2.1, X9.P2.2; no longer IRIDIUM-2.S
- net 3.3V_D2: now also X6.P2.1, X6.P2.2; no longer X1-4.S
- net 3.3V_D3: now also X8.P2.1, X8.P2.2; no longer X9-4.S
- net 5V_D1: now also X1.P3.1, X1.P3.2; no longer X4-3.S
- net 5V_D5: now also X2.P3.1, X2.P3.2; no longer X2-3.S, X5-3.S
- net 5V_D7: now also X3.P3.1, X3.P3.2, X4.P3.1, X4.P3.2; no longer X3-3.S, X6-3.S
- net BATTERY: now also X10.P2.1, X10.P2.2; no longer IRIDIUM-4.S
- net D4: now also X10.P1.1, X10.P1.2; no longer IRIDIUM-3.S
- net D6: now also X2.P2.1, X2.P2.2; no longer X2-2.S, X5-2.S
- net D8: now also X3.P2.1, X3.P2.2, X4.P2.1, X4.P2.2; no longer X3-2.S, X6-2.S
- net GND: now also X1.P1.1, X1.P1.2, X10.P3.1, X10.P3.2, X2.P1.1, X2.P1.2, X3.P1.1, X3.P1.2, X4.P1.1, X4.P1.2, X5.P1.1, X5.P1.2, X7.P1.1, X7.P1.2; no longer IRIDIUM-5.S, X1-1.S, X2-1.S, X3-1.S, X4-1.S, X5-1.S, X6-1.S, X9-1.S
- net SCL2: now also X5.P2.1, X5.P2.2; no longer X1-2.S
- net SCL3: now also X7.P2.1, X7.P2.2; no longer X9-2.S
- net SDA2: now also X6.P1.1, X6.P1.2; no longer X1-3.S
- net SDA3: now also X8.P1.1, X8.P1.2; no longer X9-3.S
Other:
- moved on the sheet: C1, C3, C4, C5, C6, C7, C8, R16
