File: Feather test/Adafruit Feather M0 Express test.sch (EAGLE design)
At the start: 45 parts, among them SW1 SPST_TACT-KMR2, U1 2MB Flash, U2 AP2112-3.3, U3 NAU7802, U4 LMV324, X1 20317, X2 32.768, X3 microUSB

Commit message: Wheatstone ordered
Parts:
- removed C10, C11: 0.1uF, SparkFun-Capacitors:0.1UF-0603-25V-(+80/-20%)
- removed C12: 1.0uF, SparkFun-Capacitors:1.0UF-0603-16V-10%
- removed J5: (no value), SparkFun-Connectors:CONN_021X02_NO_SILK
- removed JP2, JP4: (no value), SparkFun-Connectors:CONN_05NO_SILK
- removed JP5: I2C, SparkFun-Jumpers:JUMPER-SMT_3_2-NC_TRACE_SILK
- removed R10, R9: 47, SparkFun-Resistors:47OHM-0603-1/10W-1%
- removed R11, R12, R13: 100, SparkFun-Resistors:100OHM-0603-1/10W-1%
- removed U3: NAU7802, SparkFun-IC-Conversion:NAU7802SOIC
- removed U4: LMV324, SparkFun-IC-Amplifiers:LMV324
- added D1, D2: MBR120, microbuilder:DIODE-SCHOTTKYSOD-123
- added IC1: MPM3610, microbuilder:MPM3610
- added Q1: BSS138, adafruit:MOSFET-NREFLOW
- C3, C9: value 0.1uF -> 22uF; device SparkFun-Capacitors:0.1UF-0603-25V-(+80/-20%) -> microbuilder:CAP_CERAMIC0805-NOOUTLINE
- R2: value 47 -> 10K; device SparkFun-Resistors:47OHM-0603-1/10W-1% -> microbuilder:RESISTOR_0603_NOOUT
- R3: value 2.2k -> 100K; device SparkFun-Resistors:2.2KOHM-0603-1/10W-1% -> microbuilder:RESISTOR_0603_NOOUT
- R4: value 2.2k -> 10K; device SparkFun-Resistors:2.2KOHM-0603-1/10W-1% -> microbuilder:RESISTOR_0603_NOOUT
- R6: value 47 -> 100K; device SparkFun-Resistors:47OHM-0603-1/10W-1% -> microbuilder:RESISTOR_0603_NOOUT
- R8: value 100 -> 18.7K; device SparkFun-Resistors:100OHM-0603-1/10W-1% -> microbuilder:RESISTOR_0603_NOOUT
Connections:
- removed net 3.3V: JP5.2, U3.DVDD
- removed net A+: JP4.2, U4G1.+IN
- removed net A-: JP4.3, U4G3.+IN
- removed net B+: JP2.2, U4G2.+IN
- removed net B-: JP2.3, U4G4.+IN
- removed net GAIN_A-: R8.1, U4G3.-IN
- removed net GAIN_B+: R13.1, U4G2.-IN
- removed net GAIN_B-: R12.1, U4G4.-IN
- removed net INT: J5.2, U3.DRDY
- removed net N$10: R8.2, R9.1, U4G3.OUT
- removed net N$11: C10.1, U3.VBG
- removed net N$12: C3.2, R10.2, U3.VIN1P
- removed net N$13: C3.1, R9.2, U3.VIN1N
- removed net N$14: C11.2, R6.2, U3.VIN2P
- removed net N$15: C11.1, R2.2, U3.VIN2N
- removed net N$3: JP5.1, R4.2
- removed net N$4: JP5.3, R3.2
- removed net N$6: R12.2, R2.1, U4G4.OUT
- removed net N$8: R11.1, U4G1.-IN
- removed net N$9: R10.1, R11.2, U4G1.OUT
- removed net VBAT: JP3.1
- removed net VDDA: C12.1, C9.1, J5.1, JP2.5, JP4.5, U3.AVDD, U3.REFP
- new net +5V: C3.1, D2.A, IC1.OUT, JP3.3, R2.2, R6.1
- new net D12_5V: Q1.D, R2.1
- new net FB: IC1.FB, R6.2, R8.1
- new net SW: IC1.SW
- new net VIN: C9.1, IC1.IN, JP3.1, R3.1
- net +3V3: now also Q1.G, R4.2
- net D12: now also Q1.S, R4.1
- net EN: now also IC1.EN, R3.2
- net GND: now also C3.2, IC1.AGND, IC1.PGND, R8.2; no longer C10.2, C12.2, JP2.1, JP2.4, JP4.1, JP4.4, U3.AVSS, U3.DVSS, U3.REFN
- net N$1: now also C6.1, D1.C, D2.C, R1.1, U2.IN; no longer R13.2, R6.1, U4G2.OUT
- net SCL: no longer R3.1, U3.SCLK
- net SDA: no longer R4.1, U3.SDIO
- net VBUS: now also D1.A; no longer C6.1, JP3.3, R1.1, U2.IN
Other:
- note added: "BUCK DC/DC 12V TO 5V"
- note added: "LEVEL SHIFTING FOR SDI-12 (D12)"
- note removed: "154N"
- note removed: "7-bit unshifted I2C address: 0x2A"
- note removed: "A+"
- note removed: "A-"
- note removed: "B+"
- note removed: "B-"
- note removed: "Black"
- note removed: "Common Load Cell Colors:"
- note removed: "Cut jumper to remove resistors from I2C bus"
- note removed: "E+"
- note removed: "E-"
- note removed: "Green or Blue"
- note removed: "NAU7802"
- note removed: "Red"
- note removed: "Shield"
- note removed: "White"
- note removed: "Yellow"
- moved on the sheet: C3, C9
