File: DCDC/DC-DC_v3.brd (EAGLE design)
At the start: 50.8 x 27.9 mm, 16 parts, among them J2 1X2-3.5MM, J3 1X2-3.5MM, J4 1X2-3.5MM, J5 1X2-3.5MM, J7 1725698, U1 173010535, U4 173010535, U5 173010535

Commit message: Flamingo order
Parts:
- moved J2 1.91 mm to (14.0, 3.81)
- moved J3 1.27 mm to (22.2, 3.81)
- moved J4 0.64 mm to (30.5, 3.81)
Routing:
- net 3V3: track 47.2 -> 46.4 mm
- net 5V: track 35.8 -> 35.3 mm
Changed lines of the file:
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@@
 <dimension x1="0" y1="25.4" x2="50.8" y2="25.4" x3="25.4" y3="38.1" textsize="1.27" textratio="15" layer="47" unit="inch" visible="yes"/>
 <dimension x1="0" y1="25.4" x2="48.26" y2="25.4" x3="24.13" y3="33.02" textsize="1.27" textratio="15" layer="47" unit="inch" visible="yes"/>
-<text x="10.16" y="1.27" size="1.016" layer="22" rot="MR0" align="center">3V3</text>
-<text x="19.05" y="1.27" size="1.016" layer="22" rot="MR0" align="center">5V</text>
-<text x="22.86" y="1.27" size="1.016" layer="22" rot="MR0" align="center">GND</text>
-<text x="27.94" y="1.27" size="1.016" layer="22" rot="MR0" align="center">12V</text>
+<text x="12.065" y="1.27" size="1.016" layer="22" rot="MR0" align="center">3V3</text>
+<text x="20.32" y="1.27" size="1.016" layer="22" rot="MR0" align="center">5V</text>
+<text x="24.13" y="1.27" size="1.016" layer="22" rot="MR0" align="center">GND</text>
+<text x="28.575" y="1.27" size="1.016" layer="22" rot="MR0" align="center">12V</text>
 <text x="36.83" y="1.27" size="1.016" layer="22" rot="MR0" align="center">VIN</text>
-<text x="13.97" y="1.27" size="1.016" layer="22" rot="MR0" align="center">GND</text>
-<text x="31.75" y="1.27" size="1.016" layer="22" rot="MR0" align="center">GND</text>
+<text x="15.875" y="1.27" size="1.016" layer="22" rot="MR0" align="center">GND</text>
+<text x="32.385" y="1.27" size="1.016" layer="22" rot="MR0" align="center">GND</text>
 <text x="40.64" y="1.27" size="1.016" layer="22" rot="MR0" align="center">GND</text>
 <text x="43.18" y="7.62" size="1.016" layer="21" rot="R65" align="center">GND</text>
@@
 john.hulth@geo.uio.no</text>
 <text x="43.18" y="20.32" size="1.016" layer="21" rot="R65" align="center">MAIN</text>
-<text x="10.16" y="1.27" size="1.016" layer="21" align="center">3V3</text>
-<text x="19.05" y="1.27" size="1.016" layer="21" align="center">5V</text>
-<text x="22.86" y="1.27" size="1.016" layer="21" align="center">GND</text>
-<text x="27.94" y="1.27" size="1.016" layer="21" align="center">12V</text>
+<text x="12.065" y="1.27" size="1.016" layer="21" align="center">3V3</text>
+<text x="20.32" y="1.27" size="1.016" layer="21" align="center">5V</text>
+<text x="24.13" y="1.27" size="1.016" layer="21" align="center">GND</text>
+<text x="28.575" y="1.27" size="1.016" layer="21" align="center">12V</text>
 <text x="36.83" y="1.27" size="1.016" layer="21" align="center">VIN</text>
-<text x="13.97" y="1.27" size="1.016" layer="21" align="center">GND</text>
-<text x="31.75" y="1.27" size="1.016" layer="21" align="center">GND</text>
+<text x="15.875" y="1.27" size="1.016" layer="21" align="center">GND</text>
+<text x="32.385" y="1.27" size="1.016" layer="21" align="center">GND</text>
 <text x="40.64" y="1.27" size="1.016" layer="21" align="center">GND</text>
 <text x="45.72" y="7.62" size="1.016" layer="22" rot="MR0" align="center-left">GND</text>
@@
 <attribute name="MPN" value="173010535" x="24.765" y="14.605" size="1.778" layer="27" rot="R270" display="off"/>
 </element>
-<element name="J2" library="adafruit" library_urn="urn:adsk.eagle:library:420" package="1X2-3.5MM" package3d_urn="urn:adsk.eagle:package:6240635/1" value="1X2-3.5MM" x="12.065" y="3.81" smashed="yes" rot="R180"/>
-<element name="J3" library="adafruit" library_urn="urn:adsk.eagle:library:420" package="1X2-3.5MM" package3d_urn="urn:adsk.eagle:package:6240635/1" value="1X2-3.5MM" x="20.955" y="3.81" smashed="yes" rot="R180"/>
-<element name="J4" library="adafruit" library_urn="urn:adsk.eagle:library:420" package="1X2-3.5MM" package3d_urn="urn:adsk.eagle:package:6240635/1" value="1X2-3.5MM" x="29.845" y="3.81" smashed="yes" rot="R180"/>
+<element name="J2" library="adafruit" library_urn="urn:adsk.eagle:library:420" package="1X2-3.5MM" package3d_urn="urn:adsk.eagle:package:6240635/1" value="1X2-3.5MM" x="13.97" y="3.81" smashed="yes" rot="R180"/>
+<element name="J3" library="adafruit" library_urn="urn:adsk.eagle:library:420" package="1X2-3.5MM" package3d_urn="urn:adsk.eagle:package:6240635/1" value="1X2-3.5MM" x="22.225" y="3.81" smashed="yes" rot="R180"/>
+<element name="J4" library="adafruit" library_urn="urn:adsk.eagle:library:420" package="1X2-3.5MM" package3d_urn="urn:adsk.eagle:package:6240635/1" value="1X2-3.5MM" x="30.48" y="3.81" smashed="yes" rot="R180"/>
 <element name="J5" library="adafruit" library_urn="urn:adsk.eagle:library:420" package="1X2-3.5MM" package3d_urn="urn:adsk.eagle:package:6240635/1" value="1X2-3.5MM" x="38.735" y="3.81" smashed="yes" rot="R180"/>
 <element name="J7" library="154N_NAU7802_TH" package="SHDR6W90P0X254_1X6_1570X620X85" value="1725698" x="47.625" y="7.62" smashed="yes" rot="R90">
@@
 <wire x1="43.18" y1="15.24" x2="47.625" y2="15.24" width="1.27" layer="1"/>
 <wire x1="40.005" y1="12.065" x2="43.18" y2="15.24" width="1.27" layer="1"/>
-<wire x1="28.045" y1="3.81" x2="28.045" y2="5.82" width="1.27" layer="16"/>
+<wire x1="28.68" y1="3.81" x2="28.68" y2="6.455" width="1.27" layer="16"/>
 <wire x1="34.29" y1="12.065" x2="36.195" y2="12.065" width="1.27" layer="16"/>
-<wire x1="28.045" y1="5.82" x2="34.29" y2="12.065" width="1.27" layer="16"/>
+<wire x1="28.68" y1="6.455" x2="34.29" y2="12.065" width="1.27" layer="16"/>
 </signal>
 <signal name="VIN">
@@
 <wire x1="41.275" y1="9.525" x2="44.45" y2="12.7" width="1.27" layer="1"/>
 <wire x1="44.45" y1="12.7" x2="47.625" y2="12.7" width="1.27" layer="1"/>
-<wire x1="19.155" y1="3.81" x2="19.155" y2="6.455" width="1.27" layer="16"/>
-<wire x1="19.155" y1="6.455" x2="24.765" y2="12.065" width="1.27" layer="16"/>
+<wire x1="20.425" y1="3.81" x2="20.425" y2="7.725" width="1.27" layer="16"/>
+<wire x1="20.425" y1="7.725" x2="24.765" y2="12.065" width="1.27" layer="16"/>
 </signal>
 <signal name="3V3">
@@
 <wire x1="42.545" y1="6.985" x2="45.72" y2="10.16" width="1.27" layer="1"/>
 <wire x1="45.72" y1="10.16" x2="47.625" y2="10.16" width="1.27" layer="1"/>
-<wire x1="10.265" y1="3.81" x2="10.265" y2="8.995" width="1.27" layer="16"/>
-<wire x1="10.265" y1="8.995" x2="13.335" y2="12.065" width="1.27" layer="16"/>
+<wire x1="12.17" y1="3.81" x2="12.17" y2="10.9" width="1.27" layer="16"/>
+<wire x1="12.17" y1="10.9" x2="13.335" y2="12.065" width="1.27" layer="16"/>
 </signal>
 <signal name="BACK-UP">
