File: DCDC/DC-DC.brd (EAGLE design)
At the start: 50.8 x 25.4 mm, 13 parts, among them J1 61300511121, U1 173010535, U4 173010535, U5 173010535, X1 22-23-2021, X2 22-23-2021, X3 22-23-2021, X4 22-23-2021

Commit message: Merry Christmas
Parts:
- renumbered J1 to J2, JP2 to JP5, JP3 to JP6, JP8 to JP1, JP9 to JP4, U$3 to U$1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
