File: SpotOn/Drone PCB/Drone PCB.brd (EAGLE design)
At the start: 148 x 380 mm, 50 parts, among them J10 PTH, J12 Serial Interface, J2 PTH, J4 PTH, J5 61300511121, J6 PTH, X2 TSW-106-07-G-D

Commit message: Lagopus 3.0 order
Parts:
- added J1: (no value), SparkFun-Connectors:1X04_NO_SILK
- added JP3: (no value), SparkFun-Connectors:1X07
- moved J3 174.7 mm to (54.6, 374.0)
- moved J4 174.7 mm to (92.7, 374.0)
- moved H7 53.4 mm to (-63.5, 269.5)
- moved H8 53.4 mm to (-43.2, 269.5)
- moved J10 53.4 mm to (-59.7, 269.5)
- moved J11 53.4 mm to (-49.5, 269.5)
- moved J12 53.4 mm to (-59.7, 306.3)
- moved U$17 53.4 mm to (-54.6, 269.9)
- moved U$18 53.4 mm to (-52.1, 269.9)
- moved U$5 53.4 mm to (-47.8, 288.8)
- moved U$6 53.4 mm to (-49.1, 286.5)
- moved U$7 53.4 mm to (-59.7, 269.9)
- moved U$8 53.4 mm to (-57.1, 269.9)
- moved U$19 53.4 mm to (-49.5, 269.7)
- moved U$20 53.4 mm to (-47.0, 269.7)
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Connections:
- new net 12V1: J1.1
- new net 3V1: JP3.7
- new net GND1: J1.4
- new net GND2: JP3.1, JP3.6
- new net PWM: JP3.2
- new net RDY: JP3.3
- new net RS_RX: J1.3
- new net RS_TX: J1.2
- new net SCL1: JP3.5
- new net SDA1: JP3.4
Routing:
- net RST: track 45.1 -> 24.9 mm
- net IRQ: track 38.0 -> 17.8 mm
- net CS: track 48.0 -> 27.8 mm
Other:
- board text added: "SBA5"
- board text added: "SCD30"
