File: 154N_NAU7802/154N_NAU7802.brd (EAGLE design)
At the start: 36.2 x 21.6 mm, 24 parts, among them J4 1725698, J5 1725698, U3 NAU7802, U4 LMV324

Commit message: Wheatstone ordered
Parts:
- removed R13: 100, SparkFun-Resistors:0603
- added R5: 100k, SparkFun-Resistors:0603
- R1, R7, R8: value 100 -> 100k
- moved R8 3.81 mm to (34.6, 12.7)
- renumbered R11 to R1, R12 to R7
Connections:
- net GAIN_A+: now also R5.1; no longer R8.1
- net GAIN_B+: now also R8.1; no longer R13.1
- net N$1: now also R8.2; no longer R13.2
- net N$10: now also R5.2; no longer R8.2

Commit message: John
Parts:
- added C1: 1.0uF, SparkFun-Capacitors:0603
- added IC1: MCP604SL, linear:SO14
Connections:
- net 3.3V: now also C1.1, IC1.4, U4.4
- net GND: now also C1.2, IC1.11
- net VDDA: no longer U4.4
Routing:
- net 3.3V: track 14.4 -> 37.3 mm, vias 1 -> 3
- net VDDA: track 66.8 -> 63.0 mm, vias 4 -> 1
- net GAIN_A-: track 18.8 -> 17.3 mm
Changed lines of the file:
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@@
 <layer number="42" name="bRestrict" color="1" fill="10" visible="yes" active="yes"/>
 <layer number="43" name="vRestrict" color="2" fill="10" visible="yes" active="yes"/>
-<layer number="44" name="Drills" color="7" fill="1" visible="yes" active="yes"/>
+<layer number="44" name="Drills" color="7" fill="1" visible="no" active="yes"/>
 <layer number="45" name="Holes" color="7" fill="1" visible="yes" active="yes"/>
 <layer number="46" name="Milling" color="3" fill="1" visible="yes" active="yes"/>
@@
 <attribute name="VALUE" x="33.147" y="12.7" size="0.6096" layer="27" font="vector" ratio="20" rot="R90" align="top-center"/>
 </element>
+<element name="C1" library="SparkFun-Capacitors" library_urn="urn:adsk.eagle:library:510" package="0603" package3d_urn="urn:adsk.eagle:package:37414/1" value="1.0uF" x="14.9225" y="2.54" smashed="yes" rot="R270">
+<attribute name="NAME" x="15.6845" y="2.54" size="0.6096" layer="25" font="vector" ratio="20" rot="R270" align="bottom-center"/>
+<attribute name="PROD_ID" value="CAP-00868" x="14.9225" y="2.54" size="1.778" layer="27" rot="R270" display="off"/>
+<attribute name="VALUE" x="14.1605" y="2.54" size="0.6096" layer="27" font="vector" ratio="20" rot="R270" align="top-center"/>
+</element>
+<element name="IC1" library="linear" library_urn="urn:adsk.eagle:library:262" package="SO14" package3d_urn="urn:adsk.eagle:package:16406/2" value="MCP604SL" x="-8.89" y="11.43" smashed="yes">
+<attribute name="NAME" x="-13.462" y="9.525" size="1.27" layer="25" rot="R90"/>
+<attribute name="POPULARITY" value="1" x="-8.89" y="11.43" size="1.778" layer="27" display="off"/>
+<attribute name="VALUE" x="-3.048" y="9.525" size="1.27" layer="27" rot="R90"/>
+</element>
 </elements>
 <signals>
@@
 <via x="33.3375" y="7.9375" extent="1-16" drill="0.35"/>
 <via x="27.94" y="11.7475" extent="1-16" drill="0.35"/>
-<via x="22.86" y="4.1275" extent="1-16" drill="0.35"/>
 <via x="23.495" y="13.335" extent="1-16" drill="0.35"/>
-<via x="19.05" y="2.54" extent="1-16" drill="0.35"/>
+<via x="17.4625" y="2.54" extent="1-16" drill="0.35"/>
 <via x="3.175" y="1.905" extent="1-16" drill="0.35"/>
 <via x="15.24" y="17.4625" extent="1-16" drill="0.35"/>
@@
 <contactref element="J1" pad="4"/>
 <via x="6.6675" y="5.715" extent="1-16" drill="0.35"/>
-<via x="17.145" y="6.35" extent="1-16" drill="0.35"/>
+<via x="17.145" y="6.985" extent="1-16" drill="0.35"/>
 <via x="6.0325" y="16.51" extent="1-16" drill="0.35"/>
 <contactref element="U4" pad="11"/>
 <via x="27.94" y="9.8425" extent="1-16" drill="0.35"/>
 <via x="34.925" y="5.3975" extent="1-16" drill="0.35"/>
-<via x="30.7975" y="5.3975" extent="1-16" drill="0.35"/>
+<via x="30.48" y="5.08" extent="1-16" drill="0.35"/>
 <via x="17.018" y="10.795" extent="1-16" drill="0.35"/>
 <contactref element="J5" pad="2"/>
@@
 <via x="21.1455" y="8.89" extent="1-16" drill="0.35"/>
 <via x="23.368" y="8.89" extent="1-16" drill="0.35"/>
+<contactref element="C1" pad="2"/>
+<via x="23.368" y="6.985" extent="1-16" drill="0.35"/>
+<contactref element="IC1" pad="11"/>
 <wire x1="24.13" y1="18.415" x2="24.13" y2="25.0825" width="0" layer="19" extent="1-1"/>
 <wire x1="24.13" y1="-3.4925" x2="24.13" y2="3.175" width="0" layer="19" extent="1-1"/>
+<wire x1="-8.89" y1="14.03" x2="3.175" y2="12.065" width="0" layer="19" extent="1-1"/>
 </signal>
 <signal name="SCL">
@@
 <wire x1="6.6675" y1="8.89" x2="6.0325" y2="9.525" width="0.4064" layer="16"/>
 <wire x1="6.0325" y1="9.525" x2="3.175" y2="9.525" width="0.4064" layer="16"/>
+<contactref element="U4" pad="4"/>
+<contactref element="C1" pad="1"/>
+<via x="28.575" y="5.08" extent="1-16" drill="0.35"/>
+<wire x1="28.575" y1="8.095" x2="28.575" y2="5.08" width="0.4064" layer="1"/>
+<wire x1="10.795" y1="2.54" x2="13.0175" y2="2.54" width="0.4064" layer="16"/>
+<wire x1="13.0175" y1="2.54" x2="14.9225" y2="4.445" width="0.4064" layer="16"/>
+<via x="14.9225" y="4.445" extent="1-16" drill="0.35"/>
+<wire x1="14.9225" y1="4.445" x2="14.9225" y2="3.39" width="0.4064" layer="1"/>
+<wire x1="15.5575" y1="5.08" x2="14.9225" y2="4.445" width="0.4064" layer="16"/>
+<wire x1="28.575" y1="5.08" x2="15.5575" y2="5.08" width="0.4064" layer="16"/>
+<contactref element="IC1" pad="4"/>
+<wire x1="-8.89" y1="8.83" x2="3.175" y2="9.525" width="0" layer="19" extent="1-1"/>
 </signal>
 <signal name="INT">
@@
 <contactref element="U4" pad="10"/>
 <contactref element="J3" pad="1"/>
-<via x="29.845" y="15.5575" extent="1-16" drill="0.35"/>
-<wire x1="29.845" y1="15.5575" x2="29.5275" y2="15.875" width="0.254" layer="16"/>
-<wire x1="29.5275" y1="15.875" x2="21.59" y2="15.875" width="0.254" layer="16"/>
+<via x="29.845" y="15.875" extent="1-16" drill="0.35"/>
+<wire x1="29.845" y1="15.875" x2="21.59" y2="15.875" width="0.254" layer="16"/>
 <via x="21.59" y="15.875" extent="1-16" drill="0.35"/>
 <wire x1="21.59" y1="15.875" x2="21.59" y2="18.415" width="0.254" layer="1"/>
-<wire x1="29.845" y1="15.5575" x2="29.845" y2="13.495" width="0.254" layer="1"/>
+<wire x1="29.845" y1="15.875" x2="29.845" y2="13.495" width="0.254" layer="1"/>
 <contactref element="J4" pad="6"/>
 <wire x1="21.59" y1="18.415" x2="21.59" y2="25.0825" width="0" layer="19" extent="1-1"/>
@@
 <wire x1="4.445" y1="18.415" x2="10.795" y2="18.415" width="0.4064" layer="1"/>
 <wire x1="10.795" y1="7.62" x2="10.795" y2="18.415" width="0.4064" layer="1"/>
-<wire x1="13.495" y1="7.62" x2="13.876" y2="7.62" width="0.4064" layer="1"/>
-<wire x1="13.876" y1="7.62" x2="16.0985" y2="5.3975" width="0.4064" layer="1"/>
-<contactref element="U4" pad="4"/>
-<wire x1="16.0985" y1="5.3975" x2="18.7325" y2="5.3975" width="0.4064" layer="1"/>
-<via x="18.7325" y="5.3975" extent="1-16" drill="0.35"/>
-<wire x1="18.7325" y1="5.3975" x2="26.67" y2="5.3975" width="0.4064" layer="16"/>
-<via x="28.575" y="5.3975" extent="1-16" drill="0.35"/>
-<wire x1="26.67" y1="5.3975" x2="28.575" y2="5.3975" width="0.4064" layer="16"/>
-<wire x1="28.575" y1="5.3975" x2="28.575" y2="8.095" width="0.4064" layer="1"/>
-<wire x1="26.67" y1="3.175" x2="26.67" y2="5.3975" width="0.4064" layer="1"/>
-<via x="26.67" y="5.3975" extent="1-16" drill="0.35"/>
+<wire x1="13.495" y1="7.62" x2="14.511" y2="7.62" width="0.4064" layer="1"/>
+<wire x1="14.511" y1="7.62" x2="17.4155" y2="4.7155" width="0.4064" layer="1"/>
+<wire x1="17.4155" y1="4.7155" x2="20.5435" y2="1.5875" width="0.4064" layer="1"/>
+<wire x1="20.5435" y1="1.5875" x2="26.3525" y2="1.5875" width="0.4064" layer="1"/>
 <contactref element="J5" pad="3"/>
 <contactref element="J4" pad="4"/>
+<wire x1="26.67" y1="1.905" x2="26.3525" y2="1.5875" width="0.4064" layer="1"/>
+<wire x1="26.67" y1="1.905" x2="26.67" y2="3.175" width="0.4064" layer="1"/>
 <wire x1="26.67" y1="18.415" x2="26.67" y2="25.0825" width="0" layer="19" extent="1-1"/>
 <wire x1="26.67" y1="-3.4925" x2="26.67" y2="3.175" width="0" layer="19" extent="1-1"/>
@@
 <contactref element="U4" pad="5"/>
 <contactref element="J2" pad="1"/>
-<wire x1="29.845" y1="8.095" x2="29.845" y2="6.35" width="0.254" layer="1"/>
-<via x="29.845" y="6.35" extent="1-16" drill="0.35"/>
-<wire x1="29.845" y1="6.35" x2="21.59" y2="6.35" width="0.254" layer="16"/>
-<via x="21.59" y="6.35" extent="1-16" drill="0.35"/>
-<wire x1="21.59" y1="6.35" x2="21.59" y2="3.175" width="0.254" layer="1"/>
+<wire x1="29.845" y1="8.095" x2="29.845" y2="6.0325" width="0.254" layer="1"/>
+<via x="29.845" y="6.0325" extent="1-16" drill="0.35"/>
+<via x="21.59" y="6.0325" extent="1-16" drill="0.35"/>
+<wire x1="21.59" y1="6.0325" x2="21.59" y2="3.175" width="0.254" layer="1"/>
 <contactref element="J5" pad="1"/>
+<wire x1="21.59" y1="6.0325" x2="29.845" y2="6.0325" width="0.254" layer="16"/>
 <wire x1="21.59" y1="-3.4925" x2="21.59" y2="3.175" width="0" layer="19" extent="1-1"/>
 </signal>
@@
 <contactref element="U4" pad="3"/>
 <contactref element="J2" pad="4"/>
-<wire x1="29.21" y1="3.175" x2="28.8925" y2="3.175" width="0.254" layer="1"/>
-<wire x1="28.8925" y1="3.175" x2="27.6225" y2="4.445" width="0.254" layer="1"/>
-<wire x1="27.6225" y1="4.445" x2="27.6225" y2="6.0325" width="0.254" layer="1"/>
-<wire x1="27.6225" y1="6.0325" x2="27.305" y2="6.35" width="0.254" layer="1"/>
-<wire x1="27.305" y1="6.35" x2="27.305" y2="8.095" width="0.254" layer="1"/>
+<wire x1="29.21" y1="3.175" x2="27.305" y2="5.08" width="0.254" layer="1"/>
+<wire x1="27.305" y1="5.08" x2="27.305" y2="8.095" width="0.254" layer="1"/>
 <contactref element="J5" pad="4"/>
 <wire x1="29.21" y1="-3.4925" x2="29.21" y2="3.175" width="0" layer="19" extent="1-1"/>
@@
 <signal name="GAIN_A-">
 <contactref element="U4" pad="2"/>
-<via x="25.4" y="4.445" extent="1-16" drill="0.35"/>
-<wire x1="25.4" y1="4.445" x2="33.655" y2="4.445" width="0.254" layer="16"/>
-<wire x1="34.29" y1="3.81" x2="33.655" y2="4.445" width="0.254" layer="16"/>
-<wire x1="25.4" y1="6.35" x2="26.035" y2="6.985" width="0.254" layer="1"/>
-<wire x1="26.035" y1="6.985" x2="26.035" y2="8.095" width="0.254" layer="1"/>
-<wire x1="25.4" y1="4.445" x2="25.4" y2="6.35" width="0.254" layer="1"/>
+<via x="26.035" y="6.6675" extent="1-16" drill="0.35"/>
+<wire x1="26.035" y1="6.6675" x2="32.7025" y2="6.6675" width="0.254" layer="16"/>
+<wire x1="34.29" y1="5.08" x2="32.7025" y2="6.6675" width="0.254" layer="16"/>
+<wire x1="26.035" y1="6.6675" x2="26.035" y2="8.095" width="0.254" layer="1"/>
 <wire x1="26.035" y1="9.105" x2="25.4" y2="9.74" width="0.254" layer="1"/>
 <wire x1="26.035" y1="9.105" x2="26.035" y2="8.095" width="0.254" layer="1"/>
 <contactref element="J2" pad="6"/>
-<wire x1="34.29" y1="3.175" x2="34.29" y2="3.81" width="0.254" layer="16"/>
+<wire x1="34.29" y1="3.175" x2="34.29" y2="5.08" width="0.254" layer="16"/>
 <contactref element="J5" pad="6"/>
 <contactref element="R1" pad="1"/>

Commit message: Lagopus 3.0 order
Parts:
- added IC2: NAU7802SGI, NAU7802SGI:SOIC127P600X175-16N
- added RN1: CAY16-1003F4LF, CAY16-1003F4LF:CAY16-J4
- moved IC1 41.4 mm to (6.67, -27.0)
Connections:
- new net N$16: IC1.8, IC2.5, RN1.6
- new net N$5: IC1.1, IC2.2, RN1.2
- new net N$7: IC1.7, IC2.3, RN1.4
- new net N$8: IC1.14, IC2.4, RN1.8
- net A+: now also IC1.5
- net A-: now also IC1.3
- net B+: now also IC1.10
- net B-: now also IC1.12
- net GAIN_A+: now also IC1.6, RN1.3
- net GAIN_A-: now also IC1.2, RN1.1
- net GAIN_B+: now also IC1.9, RN1.5
- net GAIN_B-: now also IC1.13, RN1.7
Routing:
- net N$7: track 0.00 -> 20.6 mm
- net N$16: track 0.00 -> 20.1 mm
- net GAIN_B+: track 9.82 -> 21.0 mm
- net GAIN_A+: track 9.54 -> 20.7 mm
- net N$5: track 0.00 -> 5.90 mm
- net GAIN_B-: track 17.5 -> 23.3 mm
- net GAIN_A-: track 17.3 -> 23.2 mm
- net N$8: track 0.00 -> 5.71 mm

Commit message: Lagopus 3 mm.
Parts:
- removed IC1: MCP604SL, linear:SO14
- removed IC2: NAU7802SGI, NAU7802SGI:SOIC127P600X175-16N
- removed RN1: CAY16-1003F4LF, CAY16-1003F4LF:CAY16-J4
Connections:
- removed net N$16: IC1.8, IC2.5, RN1.6
- removed net N$5: IC1.1, IC2.2, RN1.2
- removed net N$7: IC1.7, IC2.3, RN1.4
- removed net N$8: IC1.14, IC2.4, RN1.8
- net 3.3V: no longer IC1.4
- net A+: no longer IC1.5
- net A-: no longer IC1.3
- net B+: no longer IC1.10
- net B-: no longer IC1.12
- net GAIN_A+: no longer IC1.6, RN1.3
- net GAIN_A-: no longer IC1.2, RN1.1
- net GAIN_B+: no longer IC1.9, RN1.5
- net GAIN_B-: no longer IC1.13, RN1.7
- net GND: no longer IC1.11
Routing:
- net N$7: track 20.6 -> 0.00 mm
- net N$16: track 20.1 -> 0.00 mm
- net GAIN_B+: track 21.0 -> 9.82 mm
- net GAIN_A+: track 20.7 -> 9.54 mm
- net N$5: track 5.90 -> 0.00 mm
- net GAIN_B-: track 23.3 -> 17.5 mm
- net GAIN_A-: track 23.2 -> 17.3 mm
- net N$8: track 5.71 -> 0.00 mm
