File: Other/Adafruit QT Py.brd (EAGLE design)
At the start: 17.8 x 20.7 mm, 27 parts, among them IC3 ATSAMD21E, Q2 reset, U1 AP2112K-3.3, X6 USB TYPE C

Commit message: Lagopus 3 mm.
Parts:
- added Q1: QTPY, 154N_NAU7802_TH:QTPY
Connections:
- new net 3V: Q1.11, Q1.11C
- new net 5V: Q1.13, Q1.13C
- new net MI: Q1.9, Q1.9C
- new net MO: Q1.10, Q1.10C
- new net RX: Q1.7, Q1.7C
- new net TX: Q1.6, Q1.6C
- net A0: now also Q1.0, Q1.0C
- net A1: now also Q1.1, Q1.1C
- net A2: now also Q1.2, Q1.2C
- net A3: now also Q1.3, Q1.3C
- net GND: now also Q1.12, Q1.12C
- net SCK: now also Q1.8, Q1.8C
- net SCL: now also Q1.5, Q1.5C
- net SDA: now also Q1.4, Q1.4C
