File: Other/Adafruit QT Py.sch (EAGLE design)
At the start: 24 parts, among them IC3 ATSAMD21E, Q2 reset, U1 AP2112K-3.3, X6 USB TYPE C

Commit message: Lagopus 3 mm.
Parts:
- added Q1: QTPY, 154N_NAU7802_TH:QTPY
Connections:
- new net 3V: Q1.3V
- new net 5V: Q1.5V
- new net MI: Q1.MI/A9/D9
- new net MO: Q1.MO/A10/D10
- new net RX: Q1.RX/A7/D7
- new net TX: Q1.TX/A6/D6
- net A0: now also Q1.A0/D0
- net A1: now also Q1.A1/D1
- net A2: now also Q1.A2/D2
- net A3: now also Q1.A3/D3
- net GND: now also Q1.GND
- net SCK: now also Q1.SCK/A8/D8
- net SCL: now also Q1.SCL/D5
- net SDA: now also Q1.SDA/D4
Changed lines of the file:
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@@
 <part name="SWC1" library="testpad" library_urn="urn:adsk.eagle:library:385" deviceset="TP" device="B1,27" package3d_urn="urn:adsk.eagle:package:27944/2" value="TPB1,27"/>
 <part name="U$8" library="microbuilder" deviceset="FIDUCIAL" device="_1MM"/>
+<part name="Q1" library="154N_NAU7802_TH" deviceset="QTPY" device=""/>
 </parts>
 <sheets>
@@
 </instance>
 <instance part="U$8" gate="G$1" x="236.22" y="10.16" smashed="yes"/>
+<instance part="Q1" gate="1" x="-55.88" y="127" smashed="yes">
+<attribute name="VALUE" x="-55.88" y="114.3" size="1.778" layer="96" align="center"/>
+<attribute name="NAME" x="-55.88" y="139.7" size="1.778" layer="95" align="center"/>
+</instance>
 </instances>
 <busses>
@@
 <pinref part="U2" gate="G$1" pin="VSS"/>
 <pinref part="GND4" gate="1" pin="GND"/>
+</segment>
+<segment>
+<pinref part="Q1" gate="1" pin="GND"/>
+<wire x1="-38.1" y1="132.08" x2="-33.02" y2="132.08" width="0.1524" layer="91"/>
+<label x="-33.02" y="132.08" size="1.27" layer="95" xref="yes"/>
 </segment>
 </net>
@@
 <wire x1="114.3" y1="167.64" x2="162.56" y2="167.64" width="0.1524" layer="91"/>
 </segment>
+<segment>
+<pinref part="Q1" gate="1" pin="A0/D0"/>
+<wire x1="-73.66" y1="134.62" x2="-78.74" y2="134.62" width="0.1524" layer="91"/>
+<label x="-78.74" y="134.62" size="1.27" layer="95" rot="R180" xref="yes"/>
+</segment>
 </net>
 <net name="VDDCORE" class="0">
@@
 <wire x1="162.56" y1="165.1" x2="114.3" y2="165.1" width="0.1524" layer="91"/>
 <label x="116.84" y="165.1" size="1.778" layer="95"/>
+</segment>
+<segment>
+<pinref part="Q1" gate="1" pin="A1/D1"/>
+<wire x1="-73.66" y1="132.08" x2="-78.74" y2="132.08" width="0.1524" layer="91"/>
+<label x="-78.74" y="132.08" size="1.27" layer="95" rot="R180" xref="yes"/>
 </segment>
 </net>
@@
 <label x="116.84" y="142.24" size="1.778" layer="95"/>
 </segment>
+<segment>
+<pinref part="Q1" gate="1" pin="SCK/A8/D8"/>
+<wire x1="-38.1" y1="121.92" x2="-33.02" y2="121.92" width="0.1524" layer="91"/>
+<label x="-33.02" y="121.92" size="1.27" layer="95" xref="yes"/>
+</segment>
 </net>
 <net name="A2" class="0">
@@
 <wire x1="114.3" y1="162.56" x2="162.56" y2="162.56" width="0.1524" layer="91"/>
 </segment>
+<segment>
+<pinref part="Q1" gate="1" pin="A2/D2"/>
+<wire x1="-73.66" y1="129.54" x2="-78.74" y2="129.54" width="0.1524" layer="91"/>
+<label x="-78.74" y="129.54" size="1.27" layer="95" rot="R180" xref="yes"/>
+</segment>
 </net>
 <net name="A3" class="0">
@@
 <wire x1="162.56" y1="160.02" x2="114.3" y2="160.02" width="0.1524" layer="91"/>
 </segment>
+<segment>
+<pinref part="Q1" gate="1" pin="A3/D3"/>
+<wire x1="-73.66" y1="127" x2="-78.74" y2="127" width="0.1524" layer="91"/>
+<label x="-78.74" y="127" size="1.27" layer="95" rot="R180" xref="yes"/>
+</segment>
 </net>
 <net name="SDA" class="0">
@@
 <label x="187.96" y="104.14" size="1.778" layer="95"/>
 </segment>
+<segment>
+<pinref part="Q1" gate="1" pin="SDA/D4"/>
+<wire x1="-73.66" y1="124.46" x2="-78.74" y2="124.46" width="0.1524" layer="91"/>
+<label x="-78.74" y="124.46" size="1.27" layer="95" rot="R180" xref="yes"/>
+</segment>
 </net>
 <net name="SCL" class="0">
@@
 <wire x1="208.28" y1="101.6" x2="187.96" y2="101.6" width="0.1524" layer="91"/>
 <label x="187.96" y="101.6" size="1.778" layer="95"/>
+</segment>
+<segment>
+<pinref part="Q1" gate="1" pin="SCL/D5"/>
+<wire x1="-73.66" y1="121.92" x2="-78.74" y2="121.92" width="0.1524" layer="91"/>
+<label x="-78.74" y="121.92" size="1.27" layer="95" rot="R180" xref="yes"/>
 </segment>
 </net>
@@
 </segment>
 </net>
+<net name="TX" class="0">
+<segment>
+<pinref part="Q1" gate="1" pin="TX/A6/D6"/>
+<wire x1="-73.66" y1="119.38" x2="-78.74" y2="119.38" width="0.1524" layer="91"/>
+<label x="-78.74" y="119.38" size="1.27" layer="95" rot="R180" xref="yes"/>
+</segment>
+</net>
+<net name="5V" class="0">
+<segment>
+<pinref part="Q1" gate="1" pin="5V"/>
+<wire x1="-38.1" y1="134.62" x2="-33.02" y2="134.62" width="0.1524" layer="91"/>
+<label x="-33.02" y="134.62" size="1.27" layer="95" xref="yes"/>
+</segment>
+</net>
+<net name="3V" class="0">
+<segment>
+<pinref part="Q1" gate="1" pin="3V"/>
+<wire x1="-38.1" y1="129.54" x2="-33.02" y2="129.54" width="0.1524" layer="91"/>
+<label x="-33.02" y="129.54" size="1.27" layer="95" xref="yes"/>
+</segment>
+</net>
+<net name="MO" class="0">
+<segment>
+<pinref part="Q1" gate="1" pin="MO/A10/D10"/>
+<wire x1="-38.1" y1="127" x2="-33.02" y2="127" width="0.1524" layer="91"/>
+<label x="-33.02" y="127" size="1.27" layer="95" xref="yes"/>
+</segment>
+</net>
+<net name="MI" class="0">
+<segment>
+<pinref part="Q1" gate="1" pin="MI/A9/D9"/>
+<wire x1="-38.1" y1="124.46" x2="-33.02" y2="124.46" width="0.1524" layer="91"/>
+<label x="-33.02" y="124.46" size="1.27" layer="95" xref="yes"/>
+</segment>
+</net>
+<net name="RX" class="0">
+<segment>
+<pinref part="Q1" gate="1" pin="RX/A7/D7"/>
+<wire x1="-38.1" y1="119.38" x2="-33.02" y2="119.38" width="0.1524" layer="91"/>
+<label x="-33.02" y="119.38" size="1.27" layer="95" xref="yes"/>
+</segment>
+</net>
