File: Backplate/Backplate_2.brd (EAGLE design)
At the start: 224.7 x 144.7 mm, 4 parts, among them J1 1725669, J2 1725672

Commit message: adfasdfas
Parts:
- added J3: 1725698, 154N_NAU7802_TH:SHDR6W90P0X254_1X6_1570X620X85
- added J4: 1725672, Backplate_2:1725672-4-2.54
- added Q1: QTPY, 154N_NAU7802_TH:QTPY
- moved J2 231.0 mm to (124.5, 127.0)
- moved J1 190.6 mm to (96.5, 127.0)
- moved U$1 187.3 mm to (88.9, 19.7), turned to 90 degrees
- moved U$12 133.7 mm to (143.5, 109.2)
Connections:
- new net 3V3: J1.1, J4.1, Q1.11, Q1.11C
- new net BATT+: J2.2, J3.1, J3.3, J3.5
- new net BATT-: J2.1, J3.2, J3.4, J3.6
- new net GND: J1.2, J4.2, Q1.12, Q1.12C
- new net SCL: J4.4, Q1.5, Q1.5C
- new net SDA: J4.3, Q1.4, Q1.4C
- new net SOLAR+: J2.4
- new net SOLAR-: J2.3
- new net TX_A6: J1.3, Q1.6, Q1.6C
Routing:
- net BATT+: track 0.00 -> 168.6 mm
- net BATT-: track 0.00 -> 152.1 mm
- net GND: track 0.00 -> 85.5 mm
- net 3V3: track 0.00 -> 80.7 mm
- net SDA: track 0.00 -> 63.3 mm
- net SCL: track 0.00 -> 60.8 mm
- net TX_A6: track 0.00 -> 55.4 mm, vias 0 -> 1
Other:
- outline, holes or cut-outs redrawn
- board text added: "3V3"
- board text added: "BATT+"
- board text added: "BATT-"
- board text added: "GND"
- board text added: "SCL"
- board text added: "SDA"
- board text added: "SOLAR+"
- board text added: "SOLAR-"
- board text added: "TX_A6"

Commit message: kjafljah
Parts:
- added J10, J11, J8, J9: (no value), Wurth_Connectors_WR-PHD:61301221021
- added J6: 5.5x2.1mm Barrel, Backplate_2:POWER_JACK_PTH
- added U$2: BATTERY, Backplate_2:BATTERY
- added U$3: (no value), UIO-John:UIO-LOGO-BL
- added U$4, U$5, U$6, U$7: (no value), UIO-John:HIVE-LOGO
- J1: value 1725669 -> 1725672; device Backplate_2:1725669 -> Backplate_2:1725672-4-2.54
- moved J3 70.6 mm to (83.8, 77.5), turned to 0 degrees
- moved U$1 48.9 mm to (45.8, 43.0)
- moved U$12 6.35 mm to (137.2, 109.2)
- moved J4 4.02 mm to (113.0, 125.7)
- moved J1 2.84 mm to (99.1, 125.7)
- moved J2 2.84 mm to (127.0, 125.7)
- moved Q1 2.54 mm to (109.2, 69.8)
Connections:
- new net RX_A7: J1.4, Q1.7, Q1.7C
- net SOLAR+: now also J6.PWR
- net SOLAR-: now also J6.GND, J6.GNDBREAK
Routing:
- net SOLAR+: track 0.00 -> 116.1 mm
- net SOLAR-: track 0.00 -> 113.2 mm
- net RX_A7: track 0.00 -> 52.1 mm
- net BATT+: track 168.6 -> 134.2 mm
- net BATT-: track 152.1 -> 123.5 mm
- net SDA: track 63.3 -> 60.5 mm
- net SCL: track 60.8 -> 58.2 mm
- net 3V3: track 80.7 -> 83.0 mm
- net GND: track 85.5 -> 86.4 mm
- net TX_A6: track 55.4 -> 55.0 mm, vias 1 -> 0
Other:
- outline, holes or cut-outs redrawn
- board text added: "(C) 2020 john.hulth@geo.uio.no"
- board text added: "RX_A7"

Commit message: Flamingo PCB
Parts:
- moved J10 2.54 mm to (22.9, 114.3)
- moved J11 2.54 mm to (63.5, 114.3)
Routing:
- added copper zone on layer 16, net BOTTOM
- added copper zone on layer 1, net TOP
