File: Backplate/Backplate_2.sch (EAGLE design)
At the start: 4 parts, among them J1 1725669, J2 1725672

Commit message: adfasdfas
Parts:
- added J3: 1725698, 154N_NAU7802_TH:1725698
- added J4: 1725672, Backplate_2:1725672
- added Q1: QTPY, 154N_NAU7802_TH:QTPY
Connections:
- new net 3V3: J1.1, J4.1, Q1.3V
- new net BATT+: J2.2, J3.1, J3.3, J3.5
- new net BATT-: J2.1, J3.2, J3.4, J3.6
- new net GND: J1.2, J4.2, Q1.GND
- new net SCL: J4.4, Q1.SCL/D5
- new net SDA: J4.3, Q1.SDA/D4
- new net SOLAR+: J2.4
- new net SOLAR-: J2.3
- new net TX_A6: J1.3, Q1.TX/A6/D6
Other:
- moved on the sheet: J1, J2
Changed lines of the file:
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@@
 <layer number="59" name="tCarbon" color="7" fill="1" visible="no" active="no"/>
 <layer number="60" name="bCarbon" color="7" fill="1" visible="no" active="no"/>
+<layer number="61" name="stand" color="7" fill="1" visible="no" active="no"/>
 <layer number="88" name="SimResults" color="9" fill="1" visible="yes" active="yes"/>
 <layer number="89" name="SimProbes" color="9" fill="1" visible="yes" active="yes"/>
@@
 <part name="J1" library="Backplate_2" deviceset="1725669" device=""/>
 <part name="J2" library="Backplate_2" deviceset="1725672" device=""/>
+<part name="J3" library="154N_NAU7802_TH" deviceset="1725698" device=""/>
+<part name="Q1" library="154N_NAU7802_TH" deviceset="QTPY" device=""/>
+<part name="J4" library="Backplate_2" deviceset="1725672" device=""/>
 </parts>
 <sheets>
@@
 <instance part="U$12" gate="G$1" x="50.8" y="43.18" smashed="yes"/>
 <instance part="U$1" gate="G$1" x="142.24" y="33.02" smashed="yes"/>
-<instance part="J1" gate="G$1" x="30.48" y="-22.86" smashed="yes">
-<attribute name="NAME" x="46.99" y="-15.24" size="1.778" layer="95" align="center-left"/>
-<attribute name="VALUE" x="46.99" y="-17.78" size="1.778" layer="96" align="center-left"/>
-</instance>
-<instance part="J2" gate="G$1" x="93.98" y="-22.86" smashed="yes">
-<attribute name="NAME" x="110.49" y="-15.24" size="1.778" layer="95" align="center-left"/>
-<attribute name="VALUE" x="110.49" y="-17.78" size="1.778" layer="96" align="center-left"/>
+<instance part="J1" gate="G$1" x="-55.88" y="22.86" smashed="yes">
+<attribute name="NAME" x="-39.37" y="30.48" size="1.778" layer="95" align="center-left"/>
+<attribute name="VALUE" x="-39.37" y="27.94" size="1.778" layer="96" align="center-left"/>
+</instance>
+<instance part="J2" gate="G$1" x="38.1" y="2.54" smashed="yes">
+<attribute name="NAME" x="54.61" y="10.16" size="1.778" layer="95" align="center-left"/>
+<attribute name="VALUE" x="54.61" y="7.62" size="1.778" layer="96" align="center-left"/>
+</instance>
+<instance part="J3" gate="G$1" x="154.94" y="25.4" smashed="yes">
+<attribute name="NAME" x="171.45" y="33.02" size="1.778" layer="95" align="center-left"/>
+<attribute name="VALUE" x="171.45" y="30.48" size="1.778" layer="96" align="center-left"/>
+</instance>
+<instance part="Q1" gate="1" x="-48.26" y="48.26" smashed="yes">
+<attribute name="VALUE" x="-48.26" y="35.56" size="1.778" layer="96" align="center"/>
+<attribute name="NAME" x="-48.26" y="60.96" size="1.778" layer="95" align="center"/>
+</instance>
+<instance part="J4" gate="G$1" x="-55.88" y="2.54" smashed="yes">
+<attribute name="NAME" x="-39.37" y="10.16" size="1.778" layer="95" align="center-left"/>
+<attribute name="VALUE" x="-39.37" y="7.62" size="1.778" layer="96" align="center-left"/>
 </instance>
 </instances>
@@
 </busses>
 <nets>
+<net name="BATT+" class="0">
+<segment>
+<pinref part="J3" gate="G$1" pin="1"/>
+<wire x1="154.94" y1="25.4" x2="149.86" y2="25.4" width="0.1524" layer="91"/>
+<label x="149.86" y="25.4" size="1.27" layer="95" rot="R180" xref="yes"/>
+</segment>
+<segment>
+<label x="149.86" y="20.32" size="1.27" layer="95" rot="R180" xref="yes"/>
+<pinref part="J3" gate="G$1" pin="3"/>
+<wire x1="149.86" y1="20.32" x2="154.94" y2="20.32" width="0.1524" layer="91"/>
+</segment>
+<segment>
+<label x="149.86" y="15.24" size="1.27" layer="95" rot="R180" xref="yes"/>
+<pinref part="J3" gate="G$1" pin="5"/>
+<wire x1="149.86" y1="15.24" x2="154.94" y2="15.24" width="0.1524" layer="91"/>
+</segment>
+<segment>
+<pinref part="J2" gate="G$1" pin="2"/>
+<wire x1="38.1" y1="0" x2="33.02" y2="0" width="0.1524" layer="91"/>
+<label x="33.02" y="0" size="1.27" layer="95" rot="R180" xref="yes"/>
+</segment>
+</net>
+<net name="BATT-" class="0">
+<segment>
+<pinref part="J3" gate="G$1" pin="2"/>
+<wire x1="154.94" y1="22.86" x2="149.86" y2="22.86" width="0.1524" layer="91"/>
+<label x="149.86" y="22.86" size="1.27" layer="95" rot="R180" xref="yes"/>
+</segment>
+<segment>
+<label x="149.86" y="17.78" size="1.27" layer="95" rot="R180" xref="yes"/>
+<pinref part="J3" gate="G$1" pin="4"/>
+<wire x1="149.86" y1="17.78" x2="154.94" y2="17.78" width="0.1524" layer="91"/>
+</segment>
+<segment>
+<label x="149.86" y="12.7" size="1.27" layer="95" rot="R180" xref="yes"/>
+<pinref part="J3" gate="G$1" pin="6"/>
+<wire x1="149.86" y1="12.7" x2="154.94" y2="12.7" width="0.1524" layer="91"/>
+</segment>
+<segment>
+<pinref part="J2" gate="G$1" pin="1"/>
+<wire x1="38.1" y1="2.54" x2="33.02" y2="2.54" width="0.1524" layer="91"/>
+<label x="33.02" y="2.54" size="1.27" layer="95" rot="R180" xref="yes"/>
+</segment>
+</net>
+<net name="SOLAR-" class="0">
+<segment>
+<pinref part="J2" gate="G$1" pin="3"/>
+<wire x1="38.1" y1="-2.54" x2="33.02" y2="-2.54" width="0.1524" layer="91"/>
+<label x="33.02" y="-2.54" size="1.27" layer="95" rot="R180" xref="yes"/>
+</segment>
+</net>
+<net name="SOLAR+" class="0">
+<segment>
+<pinref part="J2" gate="G$1" pin="4"/>
+<wire x1="38.1" y1="-5.08" x2="33.02" y2="-5.08" width="0.1524" layer="91"/>
+<label x="33.02" y="-5.08" size="1.27" layer="95" rot="R180" xref="yes"/>
+</segment>
+</net>
+<net name="3V3" class="0">
+<segment>
+<pinref part="Q1" gate="1" pin="3V"/>
+<wire x1="-30.48" y1="50.8" x2="-25.4" y2="50.8" width="0.1524" layer="91"/>
+<label x="-25.4" y="50.8" size="1.27" layer="95" xref="yes"/>
+</segment>
+<segment>
+<wire x1="-55.88" y1="2.54" x2="-60.96" y2="2.54" width="0.1524" layer="91"/>
+<label x="-60.96" y="2.54" size="1.27" layer="95" rot="R180" xref="yes"/>
+<pinref part="J4" gate="G$1" pin="1"/>
+</segment>
+<segment>
+<wire x1="-55.88" y1="22.86" x2="-60.96" y2="22.86" width="0.1524" layer="91"/>
+<label x="-60.96" y="22.86" size="1.27" layer="95" rot="R180" xref="yes"/>
+<pinref part="J1" gate="G$1" pin="1"/>
+</segment>
+</net>
+<net name="GND" class="0">
+<segment>
+<pinref part="Q1" gate="1" pin="GND"/>
+<wire x1="-30.48" y1="53.34" x2="-25.4" y2="53.34" width="0.1524" layer="91"/>
+<label x="-25.4" y="53.34" size="1.27" layer="95" xref="yes"/>
+</segment>
+<segment>
+<wire x1="-55.88" y1="0" x2="-60.96" y2="0" width="0.1524" layer="91"/>
+<label x="-60.96" y="0" size="1.27" layer="95" rot="R180" xref="yes"/>
+<pinref part="J4" gate="G$1" pin="2"/>
+</segment>
+<segment>
+<wire x1="-55.88" y1="20.32" x2="-60.96" y2="20.32" width="0.1524" layer="91"/>
+<label x="-60.96" y="20.32" size="1.27" layer="95" rot="R180" xref="yes"/>
+<pinref part="J1" gate="G$1" pin="2"/>
+</segment>
+</net>
+<net name="SCL" class="0">
+<segment>
+<pinref part="Q1" gate="1" pin="SCL/D5"/>
+<wire x1="-66.04" y1="43.18" x2="-71.12" y2="43.18" width="0.1524" layer="91"/>
+<label x="-71.12" y="43.18" size="1.27" layer="95" rot="R180" xref="yes"/>
+</segment>
+<segment>
+<label x="-60.96" y="-5.08" size="1.27" layer="95" rot="R180" xref="yes"/>
+<wire x1="-60.96" y1="-5.08" x2="-55.88" y2="-5.08" width="0.1524" layer="91"/>
+<pinref part="J4" gate="G$1" pin="4"/>
+</segment>
+</net>
+<net name="SDA" class="0">
+<segment>
+<pinref part="Q1" gate="1" pin="SDA/D4"/>
+<wire x1="-66.04" y1="45.72" x2="-71.12" y2="45.72" width="0.1524" layer="91"/>
+<label x="-71.12" y="45.72" size="1.27" layer="95" rot="R180" xref="yes"/>
+</segment>
+<segment>
+<label x="-60.96" y="-2.54" size="1.27" layer="95" rot="R180" xref="yes"/>
+<wire x1="-60.96" y1="-2.54" x2="-55.88" y2="-2.54" width="0.1524" layer="91"/>
+<pinref part="J4" gate="G$1" pin="3"/>
+</segment>
+</net>
+<net name="TX_A6" class="0">
+<segment>
+<pinref part="Q1" gate="1" pin="TX/A6/D6"/>
+<wire x1="-66.04" y1="40.64" x2="-71.12" y2="40.64" width="0.1524" layer="91"/>
+<label x="-71.12" y="40.64" size="1.27" layer="95" rot="R180" xref="yes"/>
+</segment>
+<segment>
+<label x="-60.96" y="17.78" size="1.27" layer="95" rot="R180" xref="yes"/>
+<wire x1="-60.96" y1="17.78" x2="-55.88" y2="17.78" width="0.1524" layer="91"/>
+<pinref part="J1" gate="G$1" pin="3"/>
+</segment>
+</net>
 </nets>
 </sheet>

Commit message: kjafljah
Parts:
- added J10, J11, J8, J9: (no value), Wurth_Connectors_WR-PHD:6130XX21021_61301221021
- added J6: 5.5x2.1mm Barrel, Backplate_2:POWER_JACK
- added U$2: BATTERY, Backplate_2:BATTERY
- J1: value 1725669 -> 1725672; device Backplate_2:1725669 -> Backplate_2:1725672
Connections:
- new net RX_A7: J1.4, Q1.RX/A7/D7
- net SOLAR+: now also J6.PWR
- net SOLAR-: now also J6.GND, J6.GNDBREAK
Changed lines of the file:
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@@
 <part name="U$12" library="Backplate_2" deviceset="WASPMOTE_V1.5" device=""/>
 <part name="U$1" library="Backplate_2" deviceset="BATTERY" device=""/>
-<part name="J1" library="Backplate_2" deviceset="1725669" device=""/>
 <part name="J2" library="Backplate_2" deviceset="1725672" device=""/>
 <part name="J3" library="154N_NAU7802_TH" deviceset="1725698" device=""/>
 <part name="Q1" library="154N_NAU7802_TH" deviceset="QTPY" device=""/>
 <part name="J4" library="Backplate_2" deviceset="1725672" device=""/>
+<part name="U$2" library="Backplate_2" deviceset="BATTERY" device=""/>
+<part name="J6" library="Backplate_2" deviceset="POWER_JACK" device="" value="5.5x2.1mm Barrel"/>
+<part name="J8" library="Wurth_Connectors_WR-PHD" library_urn="urn:adsk.eagle:library:14804658" deviceset="6130XX21021_61301221021" device="" package3d_urn="urn:adsk.eagle:package:14805470/2"/>
+<part name="J9" library="Wurth_Connectors_WR-PHD" library_urn="urn:adsk.eagle:library:14804658" deviceset="6130XX21021_61301221021" device="" package3d_urn="urn:adsk.eagle:package:14805470/2"/>
+<part name="J10" library="Wurth_Connectors_WR-PHD" library_urn="urn:adsk.eagle:library:14804658" deviceset="6130XX21021_61301221021" device="" package3d_urn="urn:adsk.eagle:package:14805470/2"/>
+<part name="J11" library="Wurth_Connectors_WR-PHD" library_urn="urn:adsk.eagle:library:14804658" deviceset="6130XX21021_61301221021" device="" package3d_urn="urn:adsk.eagle:package:14805470/2"/>
+<part name="J1" library="Backplate_2" deviceset="1725672" device=""/>
 </parts>
 <sheets>
@@
 <instance part="U$12" gate="G$1" x="50.8" y="43.18" smashed="yes"/>
 <instance part="U$1" gate="G$1" x="142.24" y="33.02" smashed="yes"/>
+<instance part="J2" gate="G$1" x="38.1" y="2.54" smashed="yes">
+<attribute name="NAME" x="54.61" y="10.16" size="1.778" layer="95" align="center-left"/>
+<attribute name="VALUE" x="54.61" y="7.62" size="1.778" layer="96" align="center-left"/>
+</instance>
+<instance part="J3" gate="G$1" x="154.94" y="25.4" smashed="yes">
+<attribute name="NAME" x="171.45" y="33.02" size="1.778" layer="95" align="center-left"/>
+<attribute name="VALUE" x="171.45" y="30.48" size="1.778" layer="96" align="center-left"/>
+</instance>
+<instance part="Q1" gate="1" x="-48.26" y="48.26" smashed="yes">
+<attribute name="VALUE" x="-48.26" y="35.56" size="1.778" layer="96" align="center"/>
+<attribute name="NAME" x="-48.26" y="60.96" size="1.778" layer="95" align="center"/>
+</instance>
+<instance part="J4" gate="G$1" x="-55.88" y="2.54" smashed="yes">
+<attribute name="NAME" x="-39.37" y="10.16" size="1.778" layer="95" align="center-left"/>
+<attribute name="VALUE" x="-39.37" y="7.62" size="1.778" layer="96" align="center-left"/>
+</instance>
+<instance part="U$2" gate="G$1" x="177.8" y="33.02" smashed="yes"/>
+<instance part="J6" gate="G$1" x="203.2" y="25.4" smashed="yes" rot="R180">
+<attribute name="VALUE" x="213.36" y="15.24" size="1.778" layer="96" font="vector" rot="R180"/>
+<attribute name="NAME" x="213.36" y="25.4" size="1.778" layer="95" font="vector" rot="R180"/>
+</instance>
+<instance part="J8" gate="G$1" x="-5.08" y="134.62" smashed="yes">
+<attribute name="NAME" x="3.9" y="134.97" size="1.016" layer="95"/>
+<attribute name="VALUE" x="4.04" y="132.75" size="1.016" layer="96"/>
+</instance>
+<instance part="J9" gate="G$1" x="27.94" y="134.62" smashed="yes">
+<attribute name="NAME" x="36.92" y="134.97" size="1.016" layer="95"/>
+<attribute name="VALUE" x="37.06" y="132.75" size="1.016" layer="96"/>
+</instance>
+<instance part="J10" gate="G$1" x="-63.5" y="134.62" smashed="yes">
+<attribute name="NAME" x="-54.52" y="134.97" size="1.016" layer="95"/>
+<attribute name="VALUE" x="-54.38" y="132.75" size="1.016" layer="96"/>
+</instance>
+<instance part="J11" gate="G$1" x="-30.48" y="134.62" smashed="yes">
+<attribute name="NAME" x="-21.5" y="134.97" size="1.016" layer="95"/>
+<attribute name="VALUE" x="-21.36" y="132.75" size="1.016" layer="96"/>
+</instance>
 <instance part="J1" gate="G$1" x="-55.88" y="22.86" smashed="yes">
 <attribute name="NAME" x="-39.37" y="30.48" size="1.778" layer="95" align="center-left"/>
 <attribute name="VALUE" x="-39.37" y="27.94" size="1.778" layer="96" align="center-left"/>
-</instance>
-<instance part="J2" gate="G$1" x="38.1" y="2.54" smashed="yes">
-<attribute name="NAME" x="54.61" y="10.16" size="1.778" layer="95" align="center-left"/>
-<attribute name="VALUE" x="54.61" y="7.62" size="1.778" layer="96" align="center-left"/>
-</instance>
-<instance part="J3" gate="G$1" x="154.94" y="25.4" smashed="yes">
-<attribute name="NAME" x="171.45" y="33.02" size="1.778" layer="95" align="center-left"/>
-<attribute name="VALUE" x="171.45" y="30.48" size="1.778" layer="96" align="center-left"/>
-</instance>
-<instance part="Q1" gate="1" x="-48.26" y="48.26" smashed="yes">
-<attribute name="VALUE" x="-48.26" y="35.56" size="1.778" layer="96" align="center"/>
-<attribute name="NAME" x="-48.26" y="60.96" size="1.778" layer="95" align="center"/>
-</instance>
-<instance part="J4" gate="G$1" x="-55.88" y="2.54" smashed="yes">
-<attribute name="NAME" x="-39.37" y="10.16" size="1.778" layer="95" align="center-left"/>
-<attribute name="VALUE" x="-39.37" y="7.62" size="1.778" layer="96" align="center-left"/>
 </instance>
 </instances>
@@
 <label x="33.02" y="-2.54" size="1.27" layer="95" rot="R180" xref="yes"/>
 </segment>
+<segment>
+<wire x1="200.66" y1="22.86" x2="198.12" y2="22.86" width="0.1524" layer="91"/>
+<wire x1="198.12" y1="22.86" x2="195.58" y2="22.86" width="0.1524" layer="91"/>
+<wire x1="200.66" y1="20.32" x2="198.12" y2="20.32" width="0.1524" layer="91"/>
+<wire x1="198.12" y1="20.32" x2="198.12" y2="22.86" width="0.1524" layer="91"/>
+<junction x="198.12" y="22.86"/>
+<pinref part="J6" gate="G$1" pin="GND"/>
+<pinref part="J6" gate="G$1" pin="GNDBREAK"/>
+<label x="195.58" y="22.86" size="1.778" layer="95" rot="R180" xref="yes"/>
+</segment>
 </net>
 <net name="SOLAR+" class="0">
@@
 <label x="33.02" y="-5.08" size="1.27" layer="95" rot="R180" xref="yes"/>
 </segment>
+<segment>
+<wire x1="200.66" y1="17.78" x2="195.58" y2="17.78" width="0.1524" layer="91"/>
+<pinref part="J6" gate="G$1" pin="PWR"/>
+<label x="195.58" y="17.78" size="1.778" layer="95" rot="R180" xref="yes"/>
+</segment>
 </net>
 <net name="3V3" class="0">
@@
 <wire x1="-60.96" y1="17.78" x2="-55.88" y2="17.78" width="0.1524" layer="91"/>
 <pinref part="J1" gate="G$1" pin="3"/>
+</segment>
+</net>
+<net name="RX_A7" class="0">
+<segment>
+<wire x1="-30.48" y1="40.64" x2="-25.4" y2="40.64" width="0.1524" layer="91"/>
+<label x="-25.4" y="40.64" size="1.27" layer="95" xref="yes"/>
+<pinref part="Q1" gate="1" pin="RX/A7/D7"/>
+</segment>
+<segment>
+<label x="-60.96" y="15.24" size="1.27" layer="95" rot="R180" xref="yes"/>
+<wire x1="-60.96" y1="15.24" x2="-55.88" y2="15.24" width="0.1524" layer="91"/>
+<pinref part="J1" gate="G$1" pin="4"/>
 </segment>
 </net>
@@
 </schematic>
 </drawing>
+<compatibility>
+<note version="8.2" severity="warning">
+Since Version 8.2, EAGLE supports online libraries. The ids
+of those online libraries will not be understood (or retained)
+with this version.
+</note>
+<note version="8.3" severity="warning">
+Since Version 8.3, EAGLE supports URNs for individual library
+assets (packages, symbols, and devices). The URNs of those assets
+will not be understood (or retained) with this version.
+</note>
+<note version="8.3" severity="warning">
+Since Version 8.3, EAGLE supports the association of 3D packages
+with devices in libraries, schematics, and board files. Those 3D
+packages will not be understood (or retained) with this version.
+</note>
+</compatibility>
 </eagle>
