File: GNSS/GNSS-proto.brd (EAGLE design)
At the start: 224.7 x 144.7 mm, 7 parts, among them Q1 FEATHER_MO_ADALOGGER, Q2 FEATHER_MO_ADALOGGER, Q3 ZED_F9P, Q4 ROCK_BLOCK_9603, Q5 GV-5-MOD, U1 TSR2-2450, U5 TSR2-2433

Commit message: Flamingo PCB
Parts:
- added BASE/ROVER: EG1218, adafruit:EG1218
- added C1: 0.1uF, rcl:E2,5-6E
- added EJECT_SD: SWITCH-MOMENTARY-2PTH, SparkFun-Electromechanical:TACTILE-PTH
- added Q6: INA260, GNSS-proto:INA260
- moved U1 97.4 mm to (186.7, 109.2), turned to 270 degrees
- moved U5 95.4 mm to (175.3, 109.2), turned to 270 degrees
- moved Q5 16.7 mm to (264.2, 77.5), turned to 270 degrees
Connections:
- removed net CHARGE_PROFILE: Q5.CHG_PROFILE
- removed net GREEN_LED: Q5.GREEN
- removed net LED_FUNCTION: Q5.LED_FUNCTION
- removed net LOAD+: Q5.LOAD+1, Q5.LOAD+2, Q5.LOAD+3, Q5.LOAD+4, U1.1, U5.1
- removed net RED_LED: Q5.RED
- new net BASE: BASE/ROVER.S, Q1.A0
- new net EJECT: C1.+, EJECT_SD.3, Q1.A1
- new net ROVER: BASE/ROVER.O
- new net SCL1: Q1.A4, Q6.SCL
- new net SDA1: Q1.A3, Q6.SDA
- new net VIN+: Q5.LOAD+1, Q5.LOAD+2, Q5.LOAD+3, Q5.LOAD+4, Q6.VIN+1, Q6.VIN+2
- new net VIN-: Q6.VIN-1, Q6.VIN-2, U1.1, U5.1
- new net WAKEUP: Q1.5, Q3.INT
- net 3.3V: now also Q6.VCC
- net GND: now also BASE/ROVER.P, C1.-, EJECT_SD.1, Q6.GND
Routing:
- net VIN+: track 0.00 -> 46.9 mm
- net 3.3V: track 88.7 -> 130.4 mm
- net VIN-: track 0.00 -> 41.6 mm
- net LOAD+: track 26.7 -> 0.00 mm
- net SDA: track 28.6 -> 46.6 mm
- net EJECT: track 0.00 -> 18.0 mm
- net SCL: track 23.5 -> 38.7 mm
- net SCL1: track 0.00 -> 9.42 mm
- net BASE: track 0.00 -> 9.20 mm
- net WAKEUP: track 0.00 -> 8.67 mm
- net GND: track 26.7 -> 34.1 mm
- net SDA1: track 0.00 -> 5.61 mm
