File: GNSS/GNSS-proto.sch (EAGLE design)
At the start: 7 parts, among them Q1 FEATHER_MO_ADALOGGER, Q2 FEATHER_MO_ADALOGGER, Q3 ZED_F9P, Q4 ROCK_BLOCK_9603, Q5 GV-5-MOD, U1 TSR2-2450, U5 TSR2-2433

Commit message: Flamingo PCB
Parts:
- added BASE/ROVER: EG1218, adafruit:EG1218S
- added C1: 0.1uF, rcl:CPOL-EUE2,5-6E
- added EJECT_SD: SWITCH-MOMENTARY-2PTH, SparkFun-Electromechanical:SWITCH-MOMENTARY-2PTH
- added Q6: INA260, GNSS-proto:INA260
Connections:
- removed net CHARGE_PROFILE: Q5.CHARGE_PROFILE
- removed net GREEN_LED: Q5.GREEN
- removed net LED_FUNCTION: Q5.LED_FUNCTION
- removed net LOAD+: Q5.LOAD+, U1.VIN, U5.VIN
- removed net RED_LED: Q5.RED
- new net BASE: BASE/ROVER.S, Q1.A0
- new net EJECT: C1.+, EJECT_SD.2, Q1.A1
- new net ROVER: BASE/ROVER.O
- new net SCL1: Q1.A4, Q6.SCL
- new net SDA1: Q1.A3, Q6.SDA
- new net VIN+: Q5.LOAD+, Q6.VIN+
- new net VIN-: Q6.VIN-, U1.VIN, U5.VIN
- new net WAKEUP: Q1.5, Q3.INT
- net 3.3V: now also Q6.VCC
- net GND: now also BASE/ROVER.P, C1.-, EJECT_SD.1, Q6.GND
Other:
- note added: "DC/DC regulators"
- note added: "GNSS"
- note added: "Power monitor"
- note added: "RAWX logger"
- note added: "RTK data"
- note added: "Solar regulator"
- moved on the sheet: Q5, U1, U5
