File: SpotOn/MLX_FIGARO/MLX_FIGARO.brd (EAGLE design)
At the start: 43.2 x 15.2 mm, 5 parts, among them J2 PTH, U1 TG2600, U2 MLX90614ESF-BAA-000-TU

Commit message: Flamingo order
Parts:
- added U$3: (no value), UIO-John:UIO-LOGO-BL
Other:
- board text added: "(C) 2021 john.hulth@geo.uio.no"
- board text added: "3V3"
- board text added: "5V"
- board text added: "ANA"
- board text added: "GND"
- board text added: "SCL"
- board text added: "SDA"
Changed lines of the file:
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@@
 <drawing>
 <settings>
-<setting alwaysvectorfont="no"/>
+<setting alwaysvectorfont="yes"/>
 <setting verticaltext="up"/>
 </settings>
@@
 <dimension x1="0" y1="-1.27" x2="43.18" y2="-1.27" x3="21.59" y3="-5.08" textsize="1.778" layer="48"/>
 <dimension x1="44.45" y1="0" x2="44.45" y2="15.24" x3="49.53" y3="7.62" textsize="1.778" layer="48"/>
+<text x="20.32" y="4.445" size="1.27" layer="22" font="vector" rot="MR180">(C) 2021
+john.hulth@geo.uio.no</text>
+<text x="3.81" y="11.43" size="1.016" layer="21" align="center-left">GND</text>
+<text x="3.81" y="8.89" size="1.016" layer="21" align="center-left">3V3</text>
+<text x="3.81" y="6.35" size="1.016" layer="21" align="center-left">SDA</text>
+<text x="3.81" y="3.81" size="1.016" layer="21" align="center-left">SCL</text>
+<text x="39.37" y="11.43" size="1.016" layer="21" rot="R180" align="center-left">5V</text>
+<text x="39.37" y="8.89" size="1.016" layer="21" rot="R180" align="center-left">5V</text>
+<text x="39.37" y="6.35" size="1.016" layer="21" rot="R180" align="center-left">ANA</text>
+<text x="39.37" y="3.81" size="1.016" layer="21" rot="R180" align="center-left">GND</text>
 </plain>
 <attributes>
@@
 </element>
 <element name="U1" library="MLX_FIGARO" package="TO-5" value="TG2600" x="30.48" y="7.62" smashed="yes">
-<attribute name="NAME" x="30.480003125" y="7.61999375" size="1.27" layer="25" align="center"/>
-<attribute name="VALUE" x="30.48" y="1.269996875" size="1.27" layer="27" align="center"/>
+<attribute name="VALUE" x="30.48" y="1.269996875" size="1.27" layer="21" align="center"/>
 </element>
 <element name="U2" library="MLX_FIGARO" package="MLX90614ESFBAA000TU" value="MLX90614ESF-BAA-000-TU" x="12.7" y="7.62" smashed="yes">
@@
 <attribute name="MANUFACTURER_NAME" value="Melexis" x="-5.08" y="22.86" size="1.778" layer="27" display="off"/>
 <attribute name="MANUFACTURER_PART_NUMBER" value="MLX90614ESF-BAA-000-TU" x="-5.08" y="22.86" size="1.778" layer="27" display="off"/>
-<attribute name="NAME" x="12.7" y="7.62" size="1.27" layer="25" align="center"/>
 <attribute name="RS_PART_NUMBER" value="1942939" x="-5.08" y="22.86" size="1.778" layer="27" display="off"/>
 <attribute name="RS_PRICE-STOCK" value="http://uk.rs-online.com/web/p/products/1942939" x="-5.08" y="22.86" size="1.778" layer="27" display="off"/>
-<attribute name="VALUE" x="12.7" y="1.27" size="1.27" layer="27" align="center"/>
+<attribute name="VALUE" x="12.7" y="1.27" size="1.27" layer="21" align="center"/>
 </element>
 <element name="J1" library="SparkFun-Connectors" library_urn="urn:adsk.eagle:library:513" package="1X04_NO_SILK" package3d_urn="urn:adsk.eagle:package:38094/1" value="" x="40.64" y="11.43" smashed="yes" rot="R270">
-<attribute name="NAME" x="42.037" y="12.7" size="0.6096" layer="25" font="vector" ratio="20" rot="R270"/>
 <attribute name="PROD_ID" value="CONN-09696" x="40.64" y="11.43" size="1.778" layer="27" rot="R270" display="off"/>
 <attribute name="VALUE" x="38.608" y="12.7" size="0.6096" layer="27" font="vector" ratio="20" rot="R270"/>
 </element>
-<element name="J2" library="SparkFun-Connectors" package="1X04_NO_SILK" value="PTH" x="2.54" y="11.43" smashed="yes" rot="R270">
-<attribute name="NAME" x="3.937" y="12.7" size="0.6096" layer="25" font="vector" ratio="20" rot="R270"/>
-<attribute name="VALUE" x="0.508" y="12.7" size="0.6096" layer="27" font="vector" ratio="20" rot="R270"/>
-</element>
+<element name="J2" library="SparkFun-Connectors" package="1X04_NO_SILK" value="PTH" x="2.54" y="11.43" smashed="yes" rot="R270"/>
+<element name="U$3" library="UIO-John" package="UIO-LOGO-BL" value="" x="27.94" y="2.54" smashed="yes" rot="MR0"/>
 </elements>
 <signals>
@@
 </drawing>
 <compatibility>
+<note version="6.3" minversion="6.2.2" severity="warning">
+Since Version 6.2.2 text objects can contain more than one line,
+which will not be processed correctly with this version.
+</note>
 <note version="8.2" severity="warning">
 Since Version 8.2, EAGLE supports online libraries. The ids
