File: SpotOn/Flamingo PCB/flamingo_pcb.sch (EAGLE design)
At the start: 23 parts, among them J1 1725698, J2 ADAFRUIT_1X2-3.5MM, J3 1725672, J5 PTH, J8 PTH

Commit message: Flamingo order
Connections:
- removed net !CS: JP12.1
- removed net +3V3: JP8.15
- removed net 3.3V: J8.2, JP10.2, JP12.5, MS2.3V
- removed net D0: JP8.3
- removed net D1: JP8.2
- removed net D10: JP9.7
- removed net D11: JP9.6
- removed net D6: JP9.9
- removed net RS-IN: JP14.3
- removed net RS-OUT: JP14.2
- removed net SCK/SCL: JP10.4, JP12.4
- removed net SDI/SDA: JP10.3, JP12.2
- removed net SDO/ADR: JP12.3
- removed net USB: MS2.USB
- new net RS-RX: J3.1, JP14.2
- new net RS-TX: J3.2, JP14.3
- net 12V: now also J3.4
- net 3V3: now also J8.2, JP10.2, JP8.15, MS2.3V
- net CS: now also JP9.7
- net EN: no longer MS2.EN
- net GND: now also J3.3
- net IRQ: now also JP9.9
- net RST: now also JP9.6
- net RX: now also JP15.3, JP8.3; no longer JP15.4
- net SCL: now also JP10.4
- net SDA: now also JP10.3
- net TX: now also JP15.4, JP8.2; no longer JP15.3
- net VBAT: no longer MS2.VBAT

Commit message: Flamingo PCB radio
Connections:
- removed net N$25: MS2.!RESET
- net !RESET: now also MS2.!RESET
- net CS: now also MS2.GPIO5; no longer MS2.GPIO10
- net E: now also MS2.GPIO11; no longer MS2.GPIO5
- net IRQ: now also MS2.GPIO10; no longer MS2.GPIO6
- net RST: now also MS2.GPIO6; no longer MS2.GPIO11
