File: Ablamtometer/Ablatometer Keller 7LD.brd (EAGLE design)
At the start: 20 x 70 mm, 3 parts, among them Q1 154N_NAU7802_TH_QTPY

Commit message: lemming  v3 uploaded
Parts:
- added U$6: (no value), UIO-John:UIO-LOGO-BL
Routing:
- net GND: vias 2 -> 4
Other:
- board text added: "(C) 2022 john.hulth@geo.uio.no"
Changed lines of the file:
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@@
 <drawing>
 <settings>
-<setting alwaysvectorfont="no"/>
+<setting alwaysvectorfont="yes"/>
 <setting verticaltext="up"/>
 </settings>
@@
 <text x="4" y="84" size="1.778" layer="21" rot="R90" align="center-left">GND</text>
 <text x="8" y="84" size="1.778" layer="21" rot="R90" align="center-left">TX</text>
+<text x="-8.314" y="69.015" size="1.27" layer="22" font="vector" rot="MR90">(C) 2022
+john.hulth@geo.uio.no</text>
 </plain>
 <attributes>
@@
 <element name="U$1" library="UIO-John" package="KELLER_7LD" value="KELLER_7LD" x="0" y="40" smashed="yes"/>
 <element name="U$3" library="UIO-John" package="WIRE_PADS" value="WIRE_PADS" x="0" y="86.5" smashed="yes"/>
+<element name="U$6" library="UIO-John" package="UIO-LOGO-BL" value="" x="-6.456" y="75.22" smashed="yes" rot="MR90"/>
 </elements>
 <signals>
@@
 <contactref element="U$3" pad="GND"/>
 <wire x1="2" y1="86.5" x2="2" y2="79" width="1.016" layer="1"/>
+<via x="5" y="48" extent="1-16" drill="0.8"/>
+<via x="5" y="32" extent="1-16" drill="0.8"/>
+<wire x1="2.54" y1="40" x2="5" y2="32" width="0" layer="19" extent="1-1"/>
 </signal>
 <signal name="SCL">
@@
 </board>
 </drawing>
+<compatibility>
+<note version="6.3" minversion="6.2.2" severity="warning">
+Since Version 6.2.2 text objects can contain more than one line,
+which will not be processed correctly with this version.
+</note>
+</compatibility>
 </eagle>
