File: CR1000X/CR1000X MUX.brd (EAGLE design)
At the start: 103.1 x 63.6 mm, 42 parts, among them IC1 LTC4311_SC70, IC2 LTC4311_SC70, IC3 LTC4311_SC70, IC4 LTC4311_SC70, IC5 LTC4311_SC70, IC6 LTC4311_SC70, IC7 LTC4311_SC70, IC8 LTC4311_SC70, IC9 LTC4311_SC70, U2 TCA9548APWR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

Commit message: mammamia3 etc
Parts:
- removed J1: (no value), Wurth_Elektronik_Electromechanic_Terminal_Blocks_Connectors_rev19d:691311500018
- removed J2: (no value), Wurth_Elektronik_Electromechanic_Terminal_Blocks_Connectors_rev19d:691311500015
- removed J3: (no value), CR1000X proto:WURTH_ELEKTRONIK_ELECTROMECHANIC_TERMINAL_BLOCKS_CONNECTORS_REV19D_691311500018
- JP1, JP3: device microbuilder:1X12_ROUND -> adafruit:1X08-BIG
- moved JP1 35.9 mm to (-17.8, -5.59)
- moved JP3 35.9 mm to (17.8, -5.59), turned to 90 degrees
Connections:
- removed net 12V: J3.5
- removed net 1H: J1.1
- removed net 1L: J1.2
- removed net 2H: J1.4
- removed net 2L: J1.5
- removed net 3H: J1.10
- removed net 3L: J1.11
- removed net 4H: J1.13
- removed net 4L: J1.14
- removed net 5H: J2.1
- removed net 5L: J2.2
- removed net 5V: J3.1
- removed net 6H: J2.4
- removed net 6L: J2.5
- removed net 7H: J2.10
- removed net 7L: J2.11
- removed net 8H: J2.13
- removed net 8L: J2.14
- removed net C3: J3.9
- removed net C4: J3.10
- removed net C5: J3.12
- removed net C6: J3.13
- removed net C7: J3.15
- removed net C8: J3.16
- removed net G2: J3.6
- removed net G3: J3.11
- removed net G4: J3.18
- removed net P1: J1.16
- removed net P2: J1.18
- removed net RG1: J3.14
- removed net RG2: J3.17
- removed net SG1: J1.3
- removed net SG2: J1.6
- removed net SG3: J1.12
- removed net SG4: J1.15
- removed net SG5: J2.3
- removed net SG6: J2.6
- removed net SG7: J2.12
- removed net SG8: J2.15
- removed net SGP: J1.17
- removed net SGVX12: J1.9
- removed net SGVX34: J2.9
- removed net SW12-2: J3.4
- removed net VX1: J1.7
- removed net VX2: J1.8
- removed net VX3: J2.7
- removed net VX4: J2.8
- net 0SCL: now also JP3.2; no longer JP1.7
- net 0SDA: now also JP3.1; no longer JP1.8
- net 1SCL: now also JP3.4; no longer JP1.5
- net 1SDA: now also JP3.3; no longer JP1.6
- net 2SCL: now also JP3.6; no longer JP1.3
- net 2SDA: now also JP3.5; no longer JP1.4
- net 3SCL: now also JP3.8; no longer JP1.1
- net 3SDA: now also JP3.7; no longer JP1.2
- net 4SCL: now also JP1.2; no longer JP3.2
- net 4SDA: now also JP1.1; no longer JP3.1
- net 5SCL: now also JP1.4; no longer JP3.4
- net 5SDA: now also JP1.3; no longer JP3.3
- net 6SCL: now also JP1.6; no longer JP3.6
- net 6SDA: now also JP1.5; no longer JP3.5
- net 7SCL: now also JP1.8; no longer JP3.8
- net 7SDA: now also JP1.7; no longer JP3.7
- net GND: no longer J3.2
- net SCL: no longer J3.7
- net SDA: no longer J3.8
- net SW12-1: no longer J3.3
Other:
- board size 103.1 x 63.6 mm -> 38.1 x 20.3 mm
- board text removed: "12V"
- board text removed: "5V"
- board text removed: "C3"
- board text removed: "C4"
- board text removed: "C5"
- board text removed: "C6"
- board text removed: "C7"
- board text removed: "C8"
- board text removed: "G"
- board text removed: "RG1"
- board text removed: "RG2"
- board text removed: "SCL"
- board text removed: "SDA"
- board text removed: "SW12-1"
- board text removed: "SW12-2"
