File: CR1000X/CR1000X small.brd (EAGLE design)
At the start: 25.4 x 17.1 mm, 16 parts, among them U1 MIC5225-3.3, U3 ADXL343, X1 TMP117_WSON, X2 SHT4X_

Commit message: mammamia3 etc
Parts:
- U1: value MIC5225-3.3 -> AP2112K-3.3
Changed lines of the file:
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@@
 <drawing>
 <settings>
-<setting alwaysvectorfont="yes"/>
+<setting alwaysvectorfont="no"/>
 <setting verticaltext="up"/>
 </settings>
@@
 <attribute name="VALUE" x="17.907" y="2.413" size="0.4064" layer="27" ratio="10"/>
 </element>
-<element name="U1" library="adafruit_power" package="SOT23-5" value="MIC5225-3.3" x="15.875" y="7.62" smashed="yes">
+<element name="U1" library="adafruit_power" package="SOT23-5" value="AP2112K-3.3" x="15.875" y="7.62" smashed="yes">
 <attribute name="NAME" x="17.853" y="7.62" size="0.8128" layer="25" ratio="18"/>
 <attribute name="VALUE" x="17.853" y="6.985" size="0.4064" layer="27" ratio="10"/>
