File: CR1000X/CR1000X small.sch (EAGLE design)
At the start: 16 parts, among them U1 MIC5225-3.3, U3 ADXL343, X1 TMP117_WSON, X2 SHT4X_

Commit message: mammamia3 etc
Parts:
- U1: value MIC5225-3.3 -> AP2112K-3.3
Changed lines of the file:
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@@
 <part name="C12" library="microbuilder" deviceset="CAP_CERAMIC" device="0805-NOOUTLINE" value="10uF"/>
 <part name="GND25" library="supply1" library_urn="urn:adsk.eagle:library:371" deviceset="GND" device=""/>
-<part name="U1" library="adafruit_power" deviceset="VREG_SOT23-5" device="" value="MIC5225-3.3"/>
+<part name="U1" library="adafruit_power" deviceset="VREG_SOT23-5" device="" value="AP2112K-3.3"/>
 <part name="U$8" library="microbuilder" deviceset="3.3V" device=""/>
 </parts>
