File: Other/Adafruit-MAX31865-PCB-master/Adafruit MAX31865.brd (EAGLE design)
At the start: 25.4 x 27.9 mm, 29 parts, among them U1 MAX31865, U3 MIC5225-3.3, X1 3.5mm, X2 3.5mm

Commit message: mammamia3 etc
Parts:
- removed C1, C2: 0.1uF, microbuilder:0805-NO
- removed C3: 100nF, microbuilder:0805-NO
- removed C4, C5: 10uF, microbuilder:0805-NO
- removed D1, D2, D3: 1N4148, microbuilder:SOD-323
- removed FB1: (no value), microbuilder:0805-NO
- removed FID1, FID2: FIDUCIAL"", microbuilder:FIDUCIAL_1MM
- removed R1: 430Ω / 4300Ω 0.1%, microbuilder:0805-NO
- removed R6, R7, R8: 10K, microbuilder:0805-NO
- removed SJ1: (no value), microbuilder:SOLDERJUMPER_2WAY_OPEN_NOPASTE
- removed SJ3, SJ4: (no value), microbuilder:SOLDERJUMPER_ARROW_NOPASTE
- removed U$16: (no value), microbuilder:ADAFRUIT_3.5MM
- removed U$20, U$21: (no value), microbuilder:ADAFRUIT_5MM
- removed U$8: (no value), microbuilder:PCBFEAT-REV-040
- removed U1: MAX31865, microbuilder:QFN20_4MM_0.65MM
- removed U3: MIC5225-3.3, microbuilder:SOT23-5
Connections:
- removed net FORCE+: SJ1.3, SJ3.2, U1.5, X1.2
- removed net FORCE-: SJ4.1, U1.9, X2.1
- removed net N$1: R1.1, U1.3, U1.4
- removed net N$11: SJ1.2, U1.6
- removed net N$12: D3.A, R7.1, U1.13
- removed net N$13: D2.A, R8.1, U1.12
- removed net N$14: D1.A, R6.1, U1.11
- removed net N$2: R1.2, U1.1, U1.2
- removed net N$4: C2.1, FB1.1, U1.20
- removed net RTDIN+: C3.1, SJ3.1, U1.7, X1.1
- removed net RTDIN-: C3.2, SJ4.2, U1.8, X2.2
- net CS_5V: no longer D3.C
- net DRDY: no longer U1.18
- net GND: no longer C1.2, C2.2, C4.2, C5.2, SJ1.1, U1.10, U1.15, U1.16, U1.PAD, U3.2
- net SCLK_5V: no longer D2.C
- net SDI_5V: no longer D1.C
- net SDO: no longer U1.14
- net VDD: no longer C1.1, C5.1, FB1.2, R6.2, R7.2, R8.2, U1.19, U3.5
- net VIN: no longer C4.1, U3.1, U3.3
Routing:
- net VDD: track 43.1 -> 0.00 mm, vias 1 -> 0
- net N$14: track 21.5 -> 0.00 mm, vias 2 -> 0
- net N$12: track 21.4 -> 0.00 mm, vias 2 -> 0
- net DRDY: track 19.4 -> 0.00 mm, vias 1 -> 0
- net SDO: track 18.8 -> 0.54 mm, vias 1 -> 0
- net FORCE+: track 17.0 -> 0.00 mm
- net FORCE-: track 12.3 -> 0.00 mm
- net RTDIN-: track 11.6 -> 0.00 mm
- net N$13: track 11.6 -> 0.00 mm
- net RTDIN+: track 11.5 -> 0.00 mm
- net VIN: track 9.88 -> 0.00 mm
- net GND: track 8.61 -> 0.00 mm, vias 5 -> 0
- net N$11: track 6.16 -> 0.00 mm
- net N$1: track 5.66 -> 0.00 mm
- net N$4: track 5.13 -> 0.00 mm
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- removed copper zone on layer 1, net GND
- removed copper zone on layer 16, net GND
Other:
- board text removed: "2 Wire"
- board text removed: "2/3 Wire"
- board text removed: "2/3/4 Wire Platinum RTD Converter"
- board text removed: "24"
- board text removed: "3"
- board text removed: "Rref"
- board text removed: "Vin: 3-5VDC Vlogic: 3-5VDC"
