File: Other/Adafruit-MAX31865-PCB-master/Adafruit MAX31865.sch (EAGLE design)
At the start: 25 parts, among them U1 MAX31865, U3 MIC5225-3.3, X1 3.5mm, X2 3.5mm

Commit message: mammamia3 etc
Parts:
- removed C1, C2: 0.1uF, microbuilder:CAP_CERAMIC0805-NOOUTLINE
- removed C3: 100nF, microbuilder:CAP_CERAMIC0805-NOOUTLINE
- removed C4, C5: 10uF, microbuilder:CAP_CERAMIC0805-NOOUTLINE
- removed D1, D2, D3: 1N4148, microbuilder:DIODESOD-323
- removed FB1: (no value), microbuilder:FERRITE-0805NO
- removed FID1, FID2: FIDUCIAL"", microbuilder:FIDUCIAL""
- removed R1: 430Ω / 4300Ω 0.1%, microbuilder:RESISTOR0805_NOOUTLINE
- removed R6, R7, R8: 10K, microbuilder:RESISTOR0805_NOOUTLINE
- removed SJ1: (no value), microbuilder:SOLDERJUMPER_2WAY
- removed SJ3, SJ4: (no value), microbuilder:SOLDERJUMPER
- removed U1: MAX31865, microbuilder:TEMP_MAX31865
- removed U3: MIC5225-3.3, microbuilder:VREG_SOT23-5
Connections:
- removed net FORCE+: SJ1.3, SJ3.2, U1.FORCE+, X1.2
- removed net FORCE-: SJ4.1, U1.FORCE-, X2.1
- removed net N$1: R1.1, U1.ISENSOR, U1.REFIN-
- removed net N$11: SJ1.2, U1.FORCE2
- removed net N$12: D3.A, R7.1, U1.CS
- removed net N$13: D2.A, R8.1, U1.SCLK
- removed net N$14: D1.A, R6.1, U1.SDI
- removed net N$2: R1.2, U1.BIAS, U1.REFIN+
- removed net N$4: C2.1, FB1.P$1, U1.VDD
- removed net RTDIN+: C3.1, SJ3.1, U1.RTDIN+, X1.1
- removed net RTDIN-: C3.2, SJ4.2, U1.RTDIN-, X2.2
- net CS_5V: no longer D3.C
- net DRDY: no longer U1.DRDY
- net GND: no longer C1.2, C2.2, C4.2, C5.2, SJ1.1, U1.AGND@2, U1.ANGD@1, U1.GND, U1.PAD, U3.GND
- net SCLK_5V: no longer D2.C
- net SDI_5V: no longer D1.C
- net SDO: no longer U1.SDO
- net VDD: no longer C1.1, C5.1, FB1.P$2, R6.2, R7.2, R8.2, U1.DVDD, U3.OUT
- net VIN: no longer C4.1, U3.EN, U3.IN
Other:
- note removed: "R1 = 4x RTD resistance at 0°C (so 400 ohm for a 100 ohm RTD). Use high quality 1% or better resistors"
